File: Modules/Slim Line/Attenuator/Elektronics/Main/Single Attenuator.sch (KiCad schematic (older format))
At the start: 3 parts, among them J1 In, J2 Out

Commit message: Update
Parts:
- J1, J2: footprint (none) -> CATs_Connector_Audio_PJSeries:PJ-301-M-12
- RV1: footprint Potentiometer_Fader_THT:Potentiometer_Fader_Alps_RS__01_Dual -> CATs_Potentiometer_Fader_THT:Potentiometer_Fader_Alps_RS__01_Dual
Changed lines of the file:
@@
 F 0 "J1" H 1882 2625 50  0000 C CNN
 F 1 "In" H 1882 2534 50  0000 C CNN
-F 2 "" H 1850 2300 50  0001 C CNN
+F 2 "CATs_Connector_Audio_PJSeries:PJ-301-M-12" H 1850 2300 50  0001 C CNN
 F 3 "~" H 1850 2300 50  0001 C CNN
 	1    1850 2300
@@
 F 0 "RV1" H 2631 2596 50  0000 R CNN
 F 1 "100kB" H 2631 2505 50  0000 R CNN
-F 2 "Potentiometer_Fader_THT:Potentiometer_Fader_Alps_RS__01_Dual" H 2700 2550 50  0001 C CNN
+F 2 "CATs_Potentiometer_Fader_THT:Potentiometer_Fader_Alps_RS__01_Dual" H 2700 2550 50  0001 C CNN
 F 3 "~" H 2700 2550 50  0001 C CNN
 	1    2700 2550
@@
 F 0 "J2" H 3120 2575 50  0000 R CNN
 F 1 "Out" H 3120 2484 50  0000 R CNN
-F 2 "" H 3300 2550 50  0001 C CNN
+F 2 "CATs_Connector_Audio_PJSeries:PJ-301-M-12" H 3300 2550 50  0001 C CNN
 F 3 "~" H 3300 2550 50  0001 C CNN
 	1    3300 2550
