File: Modules/Standard Line/Baby8 Sequencer/Electronics/Main/Baby 8.kicad_pcb (KiCad board)
At the start: 2 copper layers, 68.6 x 107.3 mm, 62 parts, among them J1 Power, J10 Gate 6, J11 Gate 7, J12 Gate 8, J2 CV Out, J3 CLK In, J4 Reset, J5 Gate 1, J6 Gate 2, J7 Gate 3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

Commit message: 4Ch Mixer added
Connections:
- U3 pad 9: (no net) -> RESET
Routing:
- net RESET: track 35.3 -> 41.6 mm, vias 1 -> 2
