File: Modules/Slim Line/Buffered Multiple/Electronics/Main/Buffered Multiple Main.sch (KiCad schematic (older format))
At the start: 18 parts, among them J1 In 1, J2 Power, J3 Out 1-1, J4 Out 1-2, J5 Out 2-1, J6 Out 2-2, J7 In 2, U1 TL074

Commit message: Update
Parts:
- added C5, C6: 100nF, Capacitor_THT:C_Rect_L7.0mm_W2.5mm_P5.00mm, symbol Device:C
- added D1, D2: 1N5817, Diode_THT:D_DO-41_SOD81_P10.16mm_Horizontal, symbol Diode:1N5817
- added J8: Out 1-3, Connector_Audio_QingPu:Jack_3.5mm_QingPu_WQP-PJ324M, symbol Connector:AudioJack2_SwitchT
- added J9: Out 2-3, Connector_Audio_QingPu:Jack_3.5mm_QingPu_WQP-PJ324M, symbol Connector:AudioJack2_SwitchT
- added R7, R8: 1k, Resistor_THT:R_Axial_DIN0207_L6.3mm_D2.5mm_P2.54mm_Vertical, symbol Device:R
- added unit 3 of U1
- added unit 3 of U2
- added unit 5 of U2
- J1, J3, J4, J5, J6, J7: footprint Connector_Audio_PJSeries:PJ-324M-3 -> Connector_Audio_QingPu:Jack_3.5mm_QingPu_WQP-PJ324M
- R1, R2, R3, R4, R5, R6: footprint Resistor_THT:R_Axial_DIN0207_L6.3mm_D2.5mm_P7.62mm_Horizontal -> Resistor_THT:R_Axial_DIN0207_L6.3mm_D2.5mm_P2.54mm_Vertical
- renumbered U1 to U2
Connections:
- net +12V: now also C5.1, D1.1 (K), U2.4 (V+); no longer J2.7 (Pin_7), J2.8 (Pin_8)
- net -12V: now also C6.2, D2.2 (A), U2.11 (V-); no longer J2.15 (Pin_15), J2.16 (Pin_16)
- net GND: now also C5.2, C6.1, J8.S, J9.S
- net at J1.T, J7.TN, R1.1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: now also U1.10 (+)
- net at J7.T, R6.1: now also U2.3 (+), U2.5 (+), U2.10 (+); no longer U2.10 (+), U2.12 (+)
- new net: R4.2, U2.1, U2.2 (-)
- new net: R5.2, U2.6 (-), U2.7
- new net: R7.2, U1.8, U1.9 (-)
- new net: J8.T, R7.1
- new net: R8.2, U2.8, U2.9 (-)
- new net: J9.T, R8.1
- new net +12VA: D1.2 (A), J2.7 (Pin_7), J2.8 (Pin_8)
- new net -12VA: D2.1 (K), J2.15 (Pin_15), J2.16 (Pin_16)
Other:
- moved on the sheet: C1, C2, C3, C4, J1, J3, J4, J5, J6, J7, R1, R2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
