File: Modules/Haraldswerk/NGF-E LFO/Electronics/Front/Haraldswerk NGF-E LFO Front.kicad_pcb (KiCad board)
At the start: 2 copper layers, 20 x 128.5 mm, 10 parts

Commit message: Update
Parts:
- ? (x4): footprint Bohrungen:Bohrung_6.1mm -> Haraldswerk NGF-E LFO Front:Bohrung_6.1mm
- ? (x2): footprint Bohrungen:Bohrung_3.0mm -> Haraldswerk NGF-E LFO Front:Bohrung_3.0mm
- ?: footprint Bohrungen:Bohrung_7.2mm -> Haraldswerk NGF-E LFO Front:Bohrung_7.2mm
- ? (x2): footprint Bohrungen:Bohrung_3.2mm -> Haraldswerk NGF-E LFO Front:Bohrung_3.2mm
