File: Modules/Haraldswerk/NGF-E LFO/Electronics/Main/Haraldswerk NGF-E LFO Main.kicad_pcb (KiCad board)
At the start: 2 copper layers, 27.9 x 101.6 mm, 46 parts, among them J1 SAW_UP, J2 SAW_DOWN, J3 TRIANGLE, J4 SQUARE, J5 Power, J6 Select, Q1 BC547, T1 1k, U1 TL072, U2 TL072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

Commit message: Update
Parts:
- J1, J2, J3, J4: footprint Connector_Audio_Additional:PJ-323M -> Connector_Audio_QingPu:Jack_3.5mm_QingPu_WQP-PJ323M
- J5: footprint Eurorack Synth:Power_2x5_Vertical -> CATs_Eurosynth_Specials:Power_2x5_Vertical
- RV1: footprint Potentiometer_THT:Potentiometer_Alps_RK097_Single_Horizontal -> Potentiometer_THT_Additional:Potentiometer_AlpsAlpine_RK0971110
- moved RV1 5.68 mm to (0.00, 12.1), turned to 270 degrees
