File: Modules/Haraldswerk/NGF-E LFO/Electronics/Main/Haraldswerk NGF-E LFO Main.sch (KiCad schematic (older format))
At the start: 45 parts, among them J1 SAW_UP, J2 SAW_DOWN, J3 TRIANGLE, J4 SQUARE, J5 Power, J6 Select, Q1 BC547, T1 1k, U1 TL072, U2 TL072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

Commit message: Update
Parts:
- J1, J2, J3, J4: footprint Connector_Audio_Additional:PJ-323M -> Connector_Audio_QingPu:Jack_3.5mm_QingPu_WQP-PJ323M
- J5: footprint Eurorack Synth:Power_2x5_Vertical -> CATs_Eurosynth_Specials:Power_2x5_Vertical; symbol Eurorack~Synth:Power_2x5 -> Eurorack_Synth:Power_2x5
- RV1: footprint Potentiometer_THT:Potentiometer_Alps_RK097_Single_Horizontal -> Potentiometer_THT_Additional:Potentiometer_AlpsAlpine_RK0971110; symbol Device:R_POT -> Device_Additional:R_POT
Changed lines of the file:
@@
 $EndDescr
 $Comp
-L Device:R_POT RV1
+L Device_Additional:R_POT RV1
 U 1 1 60E7EEAA
 P 800 2150
 F 0 "RV1" H 730 2196 50  0000 R CNN
 F 1 "A100k" H 730 2105 50  0000 R CNN
-F 2 "Potentiometer_THT:Potentiometer_Alps_RK097_Single_Horizontal" H 730 2059 50  0001 R CNN
+F 2 "Potentiometer_THT_Additional:Potentiometer_AlpsAlpine_RK0971110" H 730 2059 50  0001 R CNN
 F 3 "~" H 800 2150 50  0001 C CNN
 	1    800  2150
-	1    0    0    -1
+	1    0    0    1
 $EndComp
 $Comp
@@
 F 0 "J1" H 7020 1133 50  0000 R CNN
 F 1 "SAW_UP" H 7020 1224 50  0000 R CNN
-F 2 "Connector_Audio_Additional:PJ-323M" H 7200 1200 50  0001 C CNN
+F 2 "Connector_Audio_QingPu:Jack_3.5mm_QingPu_WQP-PJ323M" H 7200 1200 50  0001 C CNN
 F 3 "~" H 7200 1200 50  0001 C CNN
 	1    7200 1200
@@
 F 0 "J2" H 8320 1933 50  0000 R CNN
 F 1 "SAW_DOWN" H 8320 2024 50  0000 R CNN
-F 2 "Connector_Audio_Additional:PJ-323M" H 8500 2000 50  0001 C CNN
+F 2 "Connector_Audio_QingPu:Jack_3.5mm_QingPu_WQP-PJ323M" H 8500 2000 50  0001 C CNN
 F 3 "~" H 8500 2000 50  0001 C CNN
 	1    8500 2000
@@
 F 0 "J4" H 6220 2733 50  0000 R CNN
 F 1 "SQUARE" H 6220 2824 50  0000 R CNN
-F 2 "Connector_Audio_Additional:PJ-323M" H 6400 2800 50  0001 C CNN
+F 2 "Connector_Audio_QingPu:Jack_3.5mm_QingPu_WQP-PJ323M" H 6400 2800 50  0001 C CNN
 F 3 "~" H 6400 2800 50  0001 C CNN
 	1    6400 2800
@@
 F 0 "J3" H 9870 933 50  0000 R CNN
 F 1 "TRIANGLE" H 9870 1024 50  0000 R CNN
-F 2 "Connector_Audio_Additional:PJ-323M" H 10050 1000 50  0001 C CNN
+F 2 "Connector_Audio_QingPu:Jack_3.5mm_QingPu_WQP-PJ323M" H 10050 1000 50  0001 C CNN
 F 3 "~" H 10050 1000 50  0001 C CNN
 	1    10050 1000
@@
 	10650 2050 10550 2050
 $Comp
-L Eurorack~Synth:Power_2x5 J5
+L Eurorack_Synth:Power_2x5 J5
 U 1 1 60F03A05
 P 1050 6850
 F 0 "J5" H 1158 7315 50  0000 C CNN
 F 1 "Power" H 1158 7224 50  0000 C CNN
-F 2 "Eurorack Synth:Power_2x5_Vertical" H 1100 6850 50  0001 C CNN
+F 2 "CATs_Eurosynth_Specials:Power_2x5_Vertical" H 1100 6850 50  0001 C CNN
 F 3 "" H 1100 6850 50  0001 C CNN
 	1    1050 6850
