File: Modules/YuSynth/Improved Steiner VCF/Electronics/Control/YuSynth Improved Steiner VCF Control.kicad_pcb (KiCad board)
At the start: 2 copper layers, 38.1 x 101.6 mm, 22 parts, among them J1 Audio In, J10 CO_CV, J11 Res, J12 SWb, J13 SWa, J2 Audio Out, J3 CV#1, J4 CV#2, J5 V/Oct, J6 SWb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

Commit message: Update
Parts:
- removed the REF** at (0.00, 0.00)
- added REF**: Hole_0.5mm, Control:Hole_0.5mm, F.Cu at (28.6, 101.8)
- added REF**: Hole_0.5mm, Control:Hole_0.5mm, F.Cu at (17.1, 101.8)
- added REF**: Hole_0.5mm, Control:Hole_0.5mm, F.Cu at (15.9, 101.8)
- added REF**: Hole_0.5mm, Control:Hole_0.5mm, F.Cu at (14.6, 101.8)
- added REF**: Hole_0.5mm, Control:Hole_0.5mm, F.Cu at (13.3, 101.8)
- added REF**: Hole_0.5mm, Control:Hole_0.5mm, F.Cu at (12.1, 101.8)
- added REF**: Hole_0.5mm, Control:Hole_0.5mm, F.Cu at (10.8, 101.8)
- added REF**: Hole_0.5mm, Control:Hole_0.5mm, F.Cu at (9.53, 101.8)
- added REF**: Hole_0.5mm, Control:Hole_0.5mm, F.Cu at (27.3, 101.8)
- added REF**: Hole_0.5mm, Control:Hole_0.5mm, F.Cu at (26.0, 101.8)
- added REF**: Hole_0.5mm, Control:Hole_0.5mm, F.Cu at (24.8, 101.8)
- added REF**: Hole_0.5mm, Control:Hole_0.5mm, F.Cu at (23.5, 101.8)
- added REF**: Hole_0.5mm, Control:Hole_0.5mm, F.Cu at (22.2, 101.8)
- added REF**: Hole_0.5mm, Control:Hole_0.5mm, F.Cu at (21.0, 101.8)
- added REF**: Hole_0.5mm, Control:Hole_0.5mm, F.Cu at (19.7, 101.8)
- added REF**: Hole_0.5mm, Control:Hole_0.5mm, F.Cu at (18.4, 101.8)
- moved J12 0.50 mm to (14.0, 103.4)
- moved J13 0.50 mm to (14.0, 112.0)
- moved SW1 0.50 mm to (19.1, 107.7)
Other:
- board size 38.1 x 101.6 mm -> 38.1 x 113.3 mm
- board text added: "JLCJLCJLCJLC"

Commit message: Update
Parts:
- removed REF** (x16): Hole_0.5mm, Control:Hole_0.5mm
- J1, J2, J3, J4, J5: footprint Connector_Audio_PJSeries:PJ-301-M-12 -> Connector_Audio_QingPu:Jack_3.5mm_QingPu_WQP-PJ301M-12
- SW1: value Schiebeschalter2x4 -> Mode
Connections:
- J10 pad 1: CO_In -> (no net)
- J10 pad 2: CO_Out -> (no net)
- J10 pad 4: CV#1 -> (no net)
- J10 pad 5: CV#2 -> (no net)
- J8 pad 1: AudioIn -> (no net)
