File: Modules/MFOS/Noise Cornucopia/Electronics/Main 1/MFOS Noise Cornucopia Main 1.kicad_pcb (KiCad board)
At the start: 2 copper layers, 29.2 x 101.6 mm, 39 parts, among them J1 Signal, J2 Power, J4 Power, Q1 2N3904, U1 TL072, U2 TL072

Commit message: Noise Update
Parts:
- R8: value 500k -> 1M

Commit message: Update
Parts:
- R2: value 10k -> 470k
