File: Modules/HAGIWO/Arduino VCO/Electronics/Main/Arduino VCO Main.kicad_pcb (KiCad board)
At the start: 2 copper layers, 29.2 x 101.6 mm, 42 parts, among them J1 Power, J2 V/Oct, J3 Inv, J4 Out, J5 Chord, P1 B100K, P2 B100K, P3 B100K, U1 MCP6001-OT

Commit message: Arduino VCO Update
Parts:
- removed D7: BAT43, Diode_SMD:D_SOD-123
- added C11: 10µ, Capacitor_Tantalum_SMD:CP_EIA-3216-18_Kemet-A, B.Cu at (25.4, 20.3)
- added C12: 100n, Capacitor_SMD:C_0402_1005Metric, B.Cu at (9.53, 84.5)
- added R13: 2k7, Resistor_SMD:R_0603_1608Metric, B.Cu at (6.99, 87.0)
- added R14: 100k, Resistor_SMD:R_0402_1005Metric, B.Cu at (21.0, 87.0)
- added R15: 1k, Resistor_SMD:R_0402_1005Metric, B.Cu at (25.4, 95.2)
- added R16: 100k, Resistor_SMD:R_0402_1005Metric, B.Cu at (21.0, 85.7)
- C10: value 4.7µ -> 100n; footprint Capacitor_SMD:C_0603_1608Metric -> Capacitor_SMD:C_0402_1005Metric
- C6: value 10n -> 3.3n; footprint Capacitor_SMD:C_0402_1005Metric -> Capacitor_SMD:C_0603_1608Metric
- C8: value 10n -> 22n
- D6: value BAT43 -> B5819W SL
- R10: value 220 -> 100k
- R5: value 499k -> 1M; footprint Resistor_SMD:R_0603_1608Metric -> Resistor_SMD:R_0402_1005Metric
- R7: value 3k9 -> 7k5
- U1: value MCP6001-OT -> TL072CDT; footprint Package_TO_SOT_SMD:SOT-23-5 -> Package_SO:SO-8_3.9x4.9mm_P1.27mm
- moved D6 71.2 mm to (22.9, 20.3), turned to 270 degrees
- moved C8 16.5 mm to (6.99, 85.1), turned to 90 degrees
- moved R7 16.0 mm to (7.62, 88.9)
- moved C6 14.0 mm to (9.53, 87.6), turned to 90 degrees
- moved R10 9.03 mm to (19.1, 86.4), turned to 90 degrees
- moved C10 8.13 mm to (19.7, 88.9)
- moved U1 5.85 mm to (14.6, 86.4), turned to 0 degrees
Connections:
- C10 pad 1: Net-(C10-Pad1) -> +12V
- C10 pad 2: Net-(C10-Pad2) -> GND
- C6 pad 2: GND -> Net-(C6-Pad2)
- D6 pad 1: +5V -> Net-(D6-Pad1)
- D6 pad 2: Net-(D6-Pad2) -> -12V
- J1 pad -12V: Net-(J1-Pad-12V) -> Net-(D6-Pad1)
- J4 pad T: Net-(C10-Pad2) -> Net-(J4-PadT)
- R10 pad 1: Net-(C10-Pad1) -> Net-(R10-Pad1)
- R10 pad 2: Net-(D6-Pad2) -> Net-(R10-Pad2)
- R5 pad 1: Net-(C6-Pad1) -> Net-(C8-Pad1)
- R6 pad 1: Net-(C6-Pad1) -> Net-(C8-Pad1)
- U1 pad 1: Net-(D6-Pad2) -> Net-(C6-Pad1)
- U1 pad 2: GND -> Net-(C6-Pad2)
- U1 pad 3: Net-(C8-Pad1) -> GND
- U1 pad 4: Net-(D6-Pad2) -> -12V
- U1 pad 5: +5V -> GND
Routing:
- net +12V: track 14.9 -> 119.5 mm, vias 0 -> 4
- net -12V: track 0.00 -> 85.1 mm, vias 0 -> 4
- net Net-(C8-Pad1): track 3.19 -> 28.4 mm
- net Net-(R10-Pad1): track 0.00 -> 16.1 mm, vias 0 -> 2
- net Net-(C6-Pad1): track 4.79 -> 20.9 mm, vias 0 -> 2
- net Net-(D6-Pad2): track 11.4 -> 0.00 mm
- net Net-(D6-Pad1): track 0.00 -> 6.99 mm
- net Net-(R10-Pad2): track 0.00 -> 4.64 mm
- net Net-(C6-Pad2): track 0.00 -> 4.34 mm
- net Net-(J1-Pad-12V): track 2.54 -> 0.00 mm
- net Net-(C10-Pad2): track 2.24 -> 0.00 mm
- net GND: track 6.10 -> 4.03 mm, vias 2 -> 1
- net +5V: track 120.3 -> 122.4 mm, vias 2 -> 3
- net Net-(C10-Pad1): track 2.01 -> 0.00 mm
- net Net-(J4-PadT): track 0.00 -> 1.87 mm

Commit message: Update
Parts:
- R5: value 1M -> 499k

Commit message: Update Arduino VCO
Parts:
- removed D5, D8, D9: BAT43, Diode_SMD:D_SOD-123
- D2, D3, D4: value BAT43 -> BAV99; footprint Diode_SMD:D_SOD-123 -> Package_TO_SOT_SMD:SOT-23
- moved D2 21.1 mm to (6.99, 92.7), turned to 270 degrees
- moved D3 19.1 mm to (6.99, 78.1), turned to 270 degrees
- moved D4 18.9 mm to (20.3, 76.8), turned to 0 degrees
Connections:
- D2 pad 1: +5V -> GND
- D2 pad 2: A7 -> +5V
- D3 pad 1: A7 -> GND
- D3 pad 2: GND -> +5V
- D4 pad 1: +5V -> GND
- D4 pad 2: A4 -> +5V
Routing:
- net +5V: track 122.4 -> 126.9 mm
- net A7: track 61.7 -> 63.0 mm
- net A4: track 59.5 -> 60.4 mm
- net A5: track 45.6 -> 46.5 mm
- net GND: vias 1 -> 2
