File: Modules/Slim Line/Rectifier/Electronics/Main/Rectifier Main.kicad_pcb (KiCad board)
At the start: 2 copper layers, 38.1 x 101.6 mm, 34 parts, among them J1 Negative HW, J2 Full Wave, J3 In, J4 Positive HW, J5 Power, U1 TL074, U2 TL072

Commit message: Update
Connections:
- C3 pad 1: +12V -> -12V
- C6 pad 2: -12V -> +12V
- U2 pad 4: +12V -> -12V
- U2 pad 5: Net-(R4-Pad1) -> GND
- U2 pad 6: GND -> Net-(R4-Pad1)
- U2 pad 8: -12V -> +12V
Routing:
- net -12V: track 77.5 -> 82.6 mm
- net Net-(R4-Pad1): track 8.51 -> 12.9 mm
Other:
- board text added: "Slimline Rectifier Main Rev. 022203"
- board text removed: "Slimline Rectifier Main Rev. 012202"
Changed lines of the file:
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@@
     (fp_line (start 4.65 0.95) (end 4.65 -0.95) (layer "F.Fab") (width 0.1))
     (pad "1" thru_hole circle (at 0 0 270) (size 1.6 1.6) (drill 0.8) (layers *.Cu *.Mask)
-      (net 1 "+12V") (pintype "passive"))
+      (net 3 "-12V") (pintype "passive"))
     (pad "2" thru_hole circle (at 5 0 270) (size 1.6 1.6) (drill 0.8) (layers *.Cu *.Mask)
       (net 2 "GND") (pintype "passive"))
@@
       (net 2 "GND") (pinfunction "+") (pintype "input"))
     (pad "4" thru_hole oval (at 0 7.62) (size 2.4 1.6) (drill 0.8) (layers *.Cu *.Mask)
-      (net 1 "+12V") (pinfunction "V-") (pintype "power_in"))
+      (net 3 "-12V") (pinfunction "V-") (pintype "power_in"))
     (pad "5" thru_hole oval (at 7.62 7.62) (size 2.4 1.6) (drill 0.8) (layers *.Cu *.Mask)
-      (net 16 "Net-(R4-Pad1)") (pinfunction "+") (pintype "input"))
+      (net 2 "GND") (pinfunction "+") (pintype "input"))
     (pad "6" thru_hole oval (at 7.62 5.08) (size 2.4 1.6) (drill 0.8) (layers *.Cu *.Mask)
-      (net 2 "GND") (pinfunction "-") (pintype "input"))
+      (net 16 "Net-(R4-Pad1)") (pinfunction "-") (pintype "input"))
     (pad "7" thru_hole oval (at 7.62 2.54) (size 2.4 1.6) (drill 0.8) (layers *.Cu *.Mask)
       (net 17 "Net-(R4-Pad2)") (pintype "output"))
     (pad "8" thru_hole oval (at 7.62 0) (size 2.4 1.6) (drill 0.8) (layers *.Cu *.Mask)
-      (net 3 "-12V") (pinfunction "V+") (pintype "power_in"))
+      (net 1 "+12V") (pinfunction "V+") (pintype "power_in"))
     (model "${KICAD6_3DMODEL_DIR}/Package_DIP.3dshapes/DIP-8_W7.62mm.wrl"
       (offset (xyz 0 0 0))
@@
       (net 2 "GND") (pintype "passive"))
     (pad "2" thru_hole circle (at 5 0 180) (size 1.6 1.6) (drill 0.8) (layers *.Cu *.Mask)
-      (net 3 "-12V") (pintype "passive"))
+      (net 1 "+12V") (pintype "passive"))
     (model "${KICAD6_3DMODEL_DIR}/Capacitor_THT.3dshapes/C_Disc_D4.3mm_W1.9mm_P5.00mm.wrl"
       (offset (xyz 0 0 0))
@@
   (gr_line (start 29.21 101.6) (end 29.21 72.39) (layer "Edge.Cuts") (width 0.05))
   (gr_line (start 38.1 0) (end 38.1 72.39) (layer "Edge.Cuts") (width 0.05))
-  (gr_text "Slimline Rectifier\nMain Rev. 012202" (at 2.54 54.61) (layer "F.SilkS")
+  (gr_text "Slimline Rectifier\nMain Rev. 022203" (at 2.54 54.61) (layer "F.SilkS")
     (effects (font (size 0.8 0.8) (thickness 0.1)) (justify left))
   )
-  (segment (start 16.51 59.73) (end 21.545 59.73) (width 0.25) (layer "F.Cu") (net 1))
-  (segment (start 24.12 59.7) (end 24.13 59.69) (width 0.25) (layer "F.Cu") (net 1))
+  (segment (start 29.195 52.08) (end 31.74 52.08) (width 0.25) (layer "F.Cu") (net 1))
   (segment (start 16.51 68.58) (end 24.13 68.58) (width 0.25) (layer "F.Cu") (net 1))
   (segment (start 24.13 25.4) (end 24.125 25.395) (width 0.25) (layer "F.Cu") (net 1))
   (segment (start 21.57 25.4) (end 21.575 25.395) (width 0.25) (layer "F.Cu") (net 1))
   (segment (start 19.05 25.4) (end 21.57 25.4) (width 0.25) (layer "F.Cu") (net 1))
-  (segment (start 21.545 59.73) (end 21.575 59.7) (width 0.25) (layer "F.Cu") (net 1))
+  (segment (start 24.14 52.08) (end 29.195 52.08) (width 0.25) (layer "F.Cu") (net 1))
+  (segment (start 31.74 52.08) (end 31.75 52.07) (width 0.25) (layer "F.Cu") (net 1))
+  (segment (start 24.13 52.07) (end 24.14 52.08) (width 0.25) (layer "F.Cu") (net 1))
   (segment (start 24.125 25.395) (end 21.575 25.395) (width 0.25) (layer "F.Cu") (net 1))
-  (segment (start 21.575 59.7) (end 24.12 59.7) (width 0.25) (layer "F.Cu") (net 1))
-  (via (at 24.13 59.69) (size 0.8) (drill 0.4) (layers "F.Cu" "B.Cu") (net 1))
+  (via (at 24.13 52.07) (size 0.8) (drill 0.4) (layers "F.Cu" "B.Cu") (net 1))
   (via (at 16.51 68.58) (size 0.8) (drill 0.4) (layers "F.Cu" "B.Cu") (net 1))
   (via (at 24.13 68.58) (size 0.8) (drill 0.4) (layers "F.Cu" "B.Cu") (net 1))
   (via (at 24.13 25.4) (size 0.8) (drill 0.4) (layers "F.Cu" "B.Cu") (net 1))
   (segment (start 16.51 81.28) (end 16.51 68.58) (width 0.25) (layer "B.Cu") (net 1))
+  (segment (start 24.13 52.07) (end 24.13 25.4) (width 0.25) (layer "B.Cu") (net 1))
   (segment (start 16.51 86.36) (end 16.51 81.28) (width 0.25) (layer "B.Cu") (net 1))
-  (segment (start 24.13 59.69) (end 24.13 25.4) (width 0.25) (layer "B.Cu") (net 1))
+  (segment (start 24.13 59.69) (end 24.13 52.07) (width 0.25) (layer "B.Cu") (net 1))
   (segment (start 24.13 68.58) (end 24.13 59.69) (width 0.25) (layer "B.Cu") (net 1))
-  (segment (start 29.195 52.08) (end 31.74 52.08) (width 0.25) (layer "F.Cu") (net 3))
-  (segment (start 26.67 52.07) (end 26.68 52.08) (width 0.25) (layer "F.Cu") (net 3))
+  (segment (start 16.51 59.73) (end 21.545 59.73) (width 0.25) (layer "F.Cu") (net 3))
   (segment (start 26.67 25.4) (end 26.675 25.395) (width 0.25) (layer "F.Cu") (net 3))
   (segment (start 26.675 25.395) (end 29.195 25.395) (width 0.25) (layer "F.Cu") (net 3))
-  (segment (start 31.74 52.08) (end 31.75 52.07) (width 0.25) (layer "F.Cu") (net 3))
+  (segment (start 26.66 59.7) (end 21.575 59.7) (width 0.25) (layer "F.Cu") (net 3))
+  (segment (start 26.67 59.69) (end 26.66 59.7) (width 0.25) (layer "F.Cu") (net 3))
   (segment (start 20.32 66.675) (end 26.67 66.675) (width 0.25) (layer "F.Cu") (net 3))
   (segment (start 29.195 25.395) (end 31.745 25.395) (width 0.25) (layer "F.Cu") (net 3))
-  (segment (start 26.68 52.08) (end 29.195 52.08) (width 0.25) (layer "F.Cu") (net 3))
+  (segment (start 21.545 59.73) (end 21.575 59.7) (width 0.25) (layer "F.Cu") (net 3))
   (segment (start 31.745 25.395) (end 31.75 25.4) (width 0.25) (layer "F.Cu") (net 3))
-  (via (at 26.67 52.07) (size 0.8) (drill 0.4) (layers "F.Cu" "B.Cu") (net 3))
+  (via (at 26.67 59.69) (size 0.8) (drill 0.4) (layers "F.Cu" "B.Cu") (net 3))
   (via (at 26.67 25.4) (size 0.8) (drill 0.4) (layers "F.Cu" "B.Cu") (net 3))
   (via (at 20.32 66.675) (size 0.8) (drill 0.4) (layers "F.Cu" "B.Cu") (net 3))
@@
   (segment (start 20.32 81.28) (end 20.32 66.675) (width 0.25) (layer "B.Cu") (net 3))
   (segment (start 20.32 86.36) (end 20.32 81.28) (width 0.25) (layer "B.Cu") (net 3))
-  (segment (start 26.67 66.675) (end 26.67 52.07) (width 0.25) (layer "B.Cu") (net 3))
+  (segment (start 26.67 66.675) (end 26.67 59.69) (width 0.25) (layer "B.Cu") (net 3))
+  (segment (start 26.67 59.69) (end 26.67 52.07) (width 0.25) (layer "B.Cu") (net 3))
   (segment (start 26.67 52.07) (end 26.67 25.4) (width 0.25) (layer "B.Cu") (net 3))
   (segment (start 17.785 33.015) (end 17.78 33.02) (width 0.25) (layer "F.Cu") (net 4))
@@
   (segment (start 5.9 36.38) (end 5.08 35.56) (width 0.25) (layer "B.Cu") (net 15))
   (segment (start 5.9 49.05) (end 5.9 36.38) (width 0.25) (layer "B.Cu") (net 15))
+  (segment (start 29.195 57.16) (end 31.76 57.16) (width 0.25) (layer "F.Cu") (net 16))
+  (segment (start 33.02 58.42) (end 33.02 62.23) (width 0.25) (layer "F.Cu") (net 16))
   (segment (start 32.385 63.5) (end 33.02 62.865) (width 0.25) (layer "F.Cu") (net 16))
   (segment (start 33.02 62.865) (end 33.02 62.23) (width 0.25) (layer "F.Cu") (net 16))
   (segment (start 29.21 63.5) (end 32.385 63.5) (width 0.25) (layer "F.Cu") (net 16))
+  (segment (start 31.76 57.16) (end 33.02 58.42) (width 0.25) (layer "F.Cu") (net 16))
   (segment (start 29.195 63.485) (end 29.21 63.5) (width 0.25) (layer "B.Cu") (net 16))
-  (segment (start 29.195 59.7) (end 29.195 63.485) (width 0.25) (layer "B.Cu") (net 16))
   (segment (start 35.56 70.485) (end 10.16 70.485) (width 0.25) (layer "F.Cu") (net 17))
   (segment (start 29.195 54.62) (end 33.01 54.62) (width 0.25) (layer "F.Cu") (net 17))
