File: Modules/Slim Line/Rectifier/Electronics/Main/Rectifier Main.kicad_sch (KiCad schematic)
At the start: 33 parts, among them J1 Negative HW, J2 Full Wave, J3 In, J4 Positive HW, J5 Power, U1 TL074, U2 TL072

Commit message: Update
Connections:
- net +12V: now also C6.2, U2.8 (V+); no longer C3.1, U2.4 (V-)
- net -12V: now also C3.1, U2.4 (V-); no longer C6.2, U2.8 (V+)
- net GND: now also U2.5 (+); no longer U2.6 (-)
- net at R4.1, R8.2: now also U2.6 (-); no longer U2.5 (+)
Other:
- moved on the sheet: C3, C6, U2C
Changed lines of the file:
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@@
     (pin "2")
   )
-  (symbol (lib_id "Device:C") (at 86.36 132.08 0) (unit 1)
-    (in_bom yes) (on_board yes) (fields_autoplaced)
-    (property "Reference" "C3" (id 0) (at 89.281 131.1715 0)
-      (effects (font (size 1.27 1.27)) (justify left))
-    )
-    (property "Value" "100n" (id 1) (at 89.281 133.9466 0)
-      (effects (font (size 1.27 1.27)) (justify left))
-    )
-    (property "Footprint" "Capacitor_THT:C_Disc_D4.3mm_W1.9mm_P5.00mm" (id 2) (at 87.3252 135.89 0)
-      (effects (font (size 1.27 1.27)) hide)
-    )
-    (property "Datasheet" "~" (id 3) (at 86.36 132.08 0)
+  (symbol (lib_id "Device:C") (at 86.36 144.78 180) (unit 1)
+    (in_bom yes) (on_board yes) (fields_autoplaced)
+    (property "Reference" "C3" (id 0) (at 89.281 143.8715 0)
+      (effects (font (size 1.27 1.27)) (justify right))
+    )
+    (property "Value" "100n" (id 1) (at 89.281 146.6466 0)
+      (effects (font (size 1.27 1.27)) (justify right))
+    )
+    (property "Footprint" "Capacitor_THT:C_Disc_D4.3mm_W1.9mm_P5.00mm" (id 2) (at 85.3948 140.97 0)
+      (effects (font (size 1.27 1.27)) hide)
+    )
+    (property "Datasheet" "~" (id 3) (at 86.36 144.78 0)
       (effects (font (size 1.27 1.27)) hide)
     )
@@
     (pin "2")
   )
-  (symbol (lib_id "Amplifier_Operational:TL072") (at 180.34 66.04 0) (unit 2)
+  (symbol (lib_id "Amplifier_Operational:TL072") (at 180.34 66.04 0) (mirror x) (unit 2)
     (in_bom yes) (on_board yes)
-    (property "Reference" "U2" (id 0) (at 180.34 62.23 0)
-      (effects (font (size 1.27 1.27)) (justify left))
-    )
-    (property "Value" "TL072" (id 1) (at 180.34 69.85 0)
+    (property "Reference" "U2" (id 0) (at 180.34 69.85 0)
+      (effects (font (size 1.27 1.27)) (justify left))
+    )
+    (property "Value" "TL072" (id 1) (at 180.34 62.23 0)
       (effects (font (size 1.27 1.27)) (justify left))
     )
@@
     (pin "T")
   )
-  (symbol (lib_id "Amplifier_Operational:TL072") (at 110.49 138.43 180) (unit 3)
+  (symbol (lib_id "Amplifier_Operational:TL072") (at 115.57 138.43 0) (unit 3)
     (in_bom yes) (on_board yes) (fields_autoplaced)
     (property "Reference" "U2" (id 0) (at 113.665 137.5215 0)
-      (effects (font (size 1.27 1.27)) (justify right))
+      (effects (font (size 1.27 1.27)) (justify left))
     )
     (property "Value" "TL072" (id 1) (at 113.665 140.2966 0)
-      (effects (font (size 1.27 1.27)) (justify right))
-    )
-    (property "Footprint" "Package_DIP:DIP-8_W7.62mm_LongPads" (id 2) (at 110.49 138.43 0)
-      (effects (font (size 1.27 1.27)) hide)
-    )
-    (property "Datasheet" "http://www.ti.com/lit/ds/symlink/tl071.pdf" (id 3) (at 110.49 138.43 0)
+      (effects (font (size 1.27 1.27)) (justify left))
+    )
+    (property "Footprint" "Package_DIP:DIP-8_W7.62mm_LongPads" (id 2) (at 115.57 138.43 0)
+      (effects (font (size 1.27 1.27)) hide)
+    )
+    (property "Datasheet" "http://www.ti.com/lit/ds/symlink/tl071.pdf" (id 3) (at 115.57 138.43 0)
       (effects (font (size 1.27 1.27)) hide)
     )
@@
     (pin "GND")
   )
-  (symbol (lib_id "Device:C") (at 86.36 144.78 0) (unit 1)
-    (in_bom yes) (on_board yes) (fields_autoplaced)
-    (property "Reference" "C6" (id 0) (at 89.281 143.8715 0)
-      (effects (font (size 1.27 1.27)) (justify left))
-    )
-    (property "Value" "100n" (id 1) (at 89.281 146.6466 0)
-      (effects (font (size 1.27 1.27)) (justify left))
-    )
-    (property "Footprint" "Capacitor_THT:C_Disc_D4.3mm_W1.9mm_P5.00mm" (id 2) (at 87.3252 148.59 0)
-      (effects (font (size 1.27 1.27)) hide)
-    )
-    (property "Datasheet" "~" (id 3) (at 86.36 144.78 0)
-      (effects (font (size 1.27 1.27)) hide)
-    )
+  (symbol (lib_id "Device:C") (at 86.36 132.08 180) (unit 1)
+    (in_bom yes) (on_board yes) (fields_autoplaced)
+    (property "Reference" "C6" (id 0) (at 89.281 131.1715 0)
+      (effects (font (size 1.27 1.27)) (justify right))
+    )
+    (property "Value" "100n" (id 1) (at 89.281 133.9466 0)
+      (effects (font (size 1.27 1.27)) (justify right))
+    )
+    (property "Footprint" "Capacitor_THT:C_Disc_D4.3mm_W1.9mm_P5.00mm" (id 2) (at 85.3948 128.27 0)
+      (effects (font (size 1.27 1.27)) hide)
+    )
+    (property "Datasheet" "~" (id 3) (at 86.36 132.08 0)
+      (effects (font (size 1.27 1.27)) hide)
+    )
