File: Modules/Standard Line/Envelope Follower/Electronics/Main/Envelope Follower Main.kicad_pcb (KiCad board)
At the start: 2 copper layers, 31.8 x 101.6 mm, 32 parts, among them J1 In, J2 Env, J3 Power, P1 A1M, U1 TL074

Commit message: Update
Parts:
- R13: value 1k -> 470
Connections:
- R13 pad 2: Net-(D4-Pad2) -> Net-(D4-Pad1)
- U1 pad 13: Net-(D4-Pad2) -> Net-(D4-Pad1)
- U1 pad 14: Net-(D4-Pad1) -> Net-(D4-Pad2)
Routing:
- net Net-(D4-Pad2): track 72.7 -> 77.9 mm
- net Net-(D4-Pad1): track 85.5 -> 80.3 mm
Other:
- board text added: "Envelope Follower Main Rev. 022203"
- board text removed: "Envelope Follower Main Rev. 012202"
Changed lines of the file:
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@@
     (property "Sheetname" "")
     (attr through_hole)
-    (fp_text reference "D1" (at 3.81 -2.12) (layer "F.SilkS")
-      (effects (font (size 1 1) (thickness 0.15)))
-    )
-    (fp_text value "1N4148" (at 3.81 2.12) (layer "F.Fab")
-      (effects (font (size 1 1) (thickness 0.15)))
-    )
-    (fp_text user "K" (at 0 -1.8) (layer "F.SilkS")
-      (effects (font (size 1 1) (thickness 0.15)))
-    )
-    (fp_text user "K" (at 0 -1.8) (layer "F.Fab")
-      (effects (font (size 1 1) (thickness 0.15)))
-    )
-    (fp_text user "${REFERENCE}" (at 4.11 0) (layer "F.Fab")
+    (fp_text reference "D1" (at 3.81 -2.12) (layer "Dwgs.User") hide
+      (effects (font (size 1 1) (thickness 0.15)))
+    )
+    (fp_text value "1N4148" (at 3.81 0) (layer "F.SilkS")
+      (effects (font (size 0.7 0.7) (thickness 0.08)))
+    )
+    (fp_text user "K" (at 0 -1.8) (layer "F.SilkS") hide
+      (effects (font (size 1 1) (thickness 0.15)))
+    )
+    (fp_text user "K" (at 0 -1.8) (layer "F.Fab") hide
+      (effects (font (size 1 1) (thickness 0.15)))
+    )
+    (fp_text user "${REFERENCE}" (at 4.11 0) (layer "F.Fab") hide
       (effects (font (size 0.8 0.8) (thickness 0.12)))
     )
@@
       (effects (font (size 1 1) (thickness 0.15)))
     )
-    (fp_text value "1k" (at 3.81 0) (layer "F.SilkS")
+    (fp_text value "470" (at 3.81 0) (layer "F.SilkS")
       (effects (font (size 1 1) (thickness 0.15)))
     )
@@
       (net 20 "Net-(R13-Pad1)") (pintype "passive"))
     (pad "2" thru_hole oval (at 7.62 0 180) (size 1.6 1.6) (drill 0.8) (layers *.Cu *.Mask)
-      (net 11 "Net-(D4-Pad2)") (pintype "passive"))
+      (net 10 "Net-(D4-Pad1)") (pintype "passive"))
     (model "${KICAD6_3DMODEL_DIR}/Resistor_THT.3dshapes/R_Axial_DIN0207_L6.3mm_D2.5mm_P7.62mm_Horizontal.wrl"
       (offset (xyz 0 0 0))
@@
       (net 2 "GND") (pinfunction "+") (pintype "input"))
     (pad "13" thru_hole oval (at 7.62 2.54) (size 2.4 1.6) (drill 0.8) (layers *.Cu *.Mask)
-      (net 11 "Net-(D4-Pad2)") (pinfunction "-") (pintype "input"))
+      (net 10 "Net-(D4-Pad1)") (pinfunction "-") (pintype "input"))
     (pad "14" thru_hole oval (at 7.62 0) (size 2.4 1.6) (drill 0.8) (layers *.Cu *.Mask)
-      (net 10 "Net-(D4-Pad1)") (pintype "output"))
+      (net 11 "Net-(D4-Pad2)") (pintype "output"))
     (model "${KICAD6_3DMODEL_DIR}/Package_DIP.3dshapes/DIP-14_W7.62mm.wrl"
       (offset (xyz 0 0 0))
@@
     (property "Sheetname" "")
     (attr through_hole)
-    (fp_text reference "D2" (at 3.81 -2.12) (layer "F.SilkS")
-      (effects (font (size 1 1) (thickness 0.15)))
-    )
-    (fp_text value "1N4148" (at 3.81 2.12) (layer "F.Fab")
-      (effects (font (size 1 1) (thickness 0.15)))
-    )
-    (fp_text user "K" (at 0 -1.8) (layer "F.SilkS")
-      (effects (font (size 1 1) (thickness 0.15)))
-    )
-    (fp_text user "${REFERENCE}" (at 4.11 0) (layer "F.Fab")
+    (fp_text reference "D2" (at 3.81 -2.12) (layer "Dwgs.User") hide
+      (effects (font (size 1 1) (thickness 0.15)))
+    )
+    (fp_text value "1N4148" (at 3.81 0) (layer "F.SilkS")
+      (effects (font (size 0.7 0.7) (thickness 0.08)))
+    )
+    (fp_text user "K" (at 0 -1.8) (layer "Dwgs.User") hide
+      (effects (font (size 1 1) (thickness 0.15)))
+    )
+    (fp_text user "${REFERENCE}" (at 4.11 0) (layer "F.Fab") hide
       (effects (font (size 0.8 0.8) (thickness 0.12)))
     )
-    (fp_text user "K" (at 0 -1.8) (layer "F.Fab")
+    (fp_text user "K" (at 0 -1.8) (layer "F.Fab") hide
       (effects (font (size 1 1) (thickness 0.15)))
     )
@@
   (gr_line (start 31.75 0) (end 31.75 101.6) (layer "Edge.Cuts") (width 0.05))
   (gr_line (start 0 101.6) (end 0 0) (layer "Edge.Cuts") (width 0.05))
-  (gr_text "Envelope Follower\nMain Rev. 012202" (at 17.145 64.135) (layer "F.SilkS")
+  (gr_text "Envelope Follower\nMain Rev. 022203" (at 17.145 64.135) (layer "F.SilkS")
     (effects (font (size 0.8 0.8) (thickness 0.1)) (justify left))
   )
@@
   (segment (start 5.08 22.225) (end 5.08 27.94) (width 0.25) (layer "B.Cu") (net 8))
   (segment (start 1.905 36.83) (end 5.08 36.83) (width 0.25) (layer "F.Cu") (net 9))
-  (segment (start 26.03 25.395) (end 26.035 25.4) (width 0.25) (layer "F.Cu") (net 10))
-  (segment (start 26.67 78.74) (end 6.985 78.74) (width 0.25) (layer "F.Cu") (net 10))
-  (segment (start 19.67 25.395) (end 26.03 25.395) (width 0.25) (layer "F.Cu") (net 10))
+  (segment (start 19.67 27.935) (end 22.22 27.935) (width 0.25) (layer "F.Cu") (net 10))
+  (segment (start 25.4 78.74) (end 6.985 78.74) (width 0.25) (layer "F.Cu") (net 10))
   (segment (start 3.81 76.2) (end 6.35 76.2) (width 0.25) (layer "F.Cu") (net 10))
   (segment (start 6.35 76.2) (end 6.985 76.835) (width 0.25) (layer "F.Cu") (net 10))
+  (segment (start 22.225 27.94) (end 25.4 27.94) (width 0.25) (layer "F.Cu") (net 10))
+  (segment (start 22.22 27.935) (end 22.225 27.94) (width 0.25) (layer "F.Cu") (net 10))
   (segment (start 6.985 76.835) (end 6.985 78.74) (width 0.25) (layer "F.Cu") (net 10))
-  (via (at 26.67 78.74) (size 0.8) (drill 0.4) (layers "F.Cu" "B.Cu") (net 10))
-  (via (at 26.035 25.4) (size 0.8) (drill 0.4) (layers "F.Cu" "B.Cu") (net 10))
-  (segment (start 26.67 26.67) (end 26.67 29.21) (width 0.25) (layer "B.Cu") (net 10))
-  (segment (start 26.67 70.485) (end 26.67 78.74) (width 0.25) (layer "B.Cu") (net 10))
-  (segment (start 26.035 26.035) (end 26.67 26.67) (width 0.25) (layer "B.Cu") (net 10))
-  (segment (start 26.67 29.21) (end 26.035 29.845) (width 0.25) (layer "B.Cu") (net 10))
-  (segment (start 26.035 69.85) (end 26.67 70.485) (width 0.25) (layer "B.Cu") (net 10))
-  (segment (start 26.035 25.4) (end 26.035 26.035) (width 0.25) (layer "B.Cu") (net 10))
-  (segment (start 26.035 29.845) (end 26.035 69.85) (width 0.25) (layer "B.Cu") (net 10))
-  (segment (start 19.67 27.935) (end 22.22 27.935) (width 0.25) (layer "F.Cu") (net 11))
+  (via (at 25.4 27.94) (size 0.8) (drill 0.4) (layers "F.Cu" "B.Cu") (net 10))
+  (via (at 25.4 78.74) (size 0.8) (drill 0.4) (layers "F.Cu" "B.Cu") (net 10))
+  (segment (start 25.4 27.94) (end 25.4 78.74) (width 0.25) (layer "B.Cu") (net 10))
+  (segment (start 26.03 25.395) (end 26.035 25.4) (width 0.25) (layer "F.Cu") (net 11))
   (segment (start 6.985 73.025) (end 6.985 71.12) (width 0.25) (layer "F.Cu") (net 11))
-  (segment (start 22.225 27.94) (end 25.4 27.94) (width 0.25) (layer "F.Cu") (net 11))
-  (segment (start 22.22 27.935) (end 22.225 27.94) (width 0.25) (layer "F.Cu") (net 11))
-  (segment (start 6.985 71.12) (end 25.4 71.12) (width 0.25) (layer "F.Cu") (net 11))
+  (segment (start 19.67 25.395) (end 26.03 25.395) (width 0.25) (layer "F.Cu") (net 11))
   (segment (start 6.35 73.66) (end 6.985 73.025) (width 0.25) (layer "F.Cu") (net 11))
+  (segment (start 6.985 71.12) (end 26.67 71.12) (width 0.25) (layer "F.Cu") (net 11))
   (segment (start 3.81 73.66) (end 6.35 73.66) (width 0.25) (layer "F.Cu") (net 11))
-  (via (at 25.4 27.94) (size 0.8) (drill 0.4) (layers "F.Cu" "B.Cu") (net 11))
-  (via (at 25.4 71.12) (size 0.8) (drill 0.4) (layers "F.Cu" "B.Cu") (net 11))
-  (segment (start 25.4 27.94) (end 25.4 71.12) (width 0.25) (layer "B.Cu") (net 11))
+  (via (at 26.67 71.12) (size 0.8) (drill 0.4) (layers "F.Cu" "B.Cu") (net 11))
+  (via (at 26.035 25.4) (size 0.8) (drill 0.4) (layers "F.Cu" "B.Cu") (net 11))
+  (segment (start 26.67 70.485) (end 26.035 69.85) (width 0.25) (layer "B.Cu") (net 11))
+  (segment (start 26.67 29.21) (end 26.67 26.67) (width 0.25) (layer "B.Cu") (net 11))
+  (segment (start 26.035 69.85) (end 26.035 29.845) (width 0.25) (layer "B.Cu") (net 11))
+  (segment (start 26.67 26.67) (end 26.035 26.035) (width 0.25) (layer "B.Cu") (net 11))
+  (segment (start 26.035 29.845) (end 26.67 29.21) (width 0.25) (layer "B.Cu") (net 11))
+  (segment (start 26.035 26.035) (end 26.035 25.4) (width 0.25) (layer "B.Cu") (net 11))
+  (segment (start 26.67 71.12) (end 26.67 70.485) (width 0.25) (layer "B.Cu") (net 11))
   (segment (start 17.78 94.615) (end 17.78 99.06) (width 0.25) (layer "F.Cu") (net 12))
   (segment (start 24.765 88.9) (end 24.13 89.535) (width 0.25) (layer "F.Cu") (net 12))
