File: Modules/Standard Line/Envelope Follower/Electronics/Main/Envelope Follower Main.kicad_sch (KiCad schematic)
At the start: 31 parts, among them J1 In, J2 Env, J3 Power, P1 A1M, U1 TL074

Commit message: Update
Parts:
- R13: value 1k -> 470
Connections:
- net at D4.1 (K), D5.2 (A): now also R13.2, U1.13 (-); no longer U1.14
- net at D4.2 (A), D5.1 (K): now also U1.14; no longer R13.2, U1.13 (-)
Other:
- moved on the sheet: D4, D5
Changed lines of the file:
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@@
     (pin "TN")
   )
-  (symbol (lib_id "Diode:1N4148") (at 231.14 76.2 180) (unit 1)
+  (symbol (lib_id "Diode:1N4148") (at 231.14 76.2 0) (unit 1)
     (in_bom yes) (on_board yes) (fields_autoplaced)
     (property "Reference" "D4" (id 0) (at 231.14 70.9635 0))
     (property "Value" "1N4148" (id 1) (at 231.14 73.7386 0))
-    (property "Footprint" "Diode_THT:D_DO-35_SOD27_P7.62mm_Horizontal" (id 2) (at 231.14 71.755 0)
+    (property "Footprint" "Diode_THT:D_DO-35_SOD27_P7.62mm_Horizontal" (id 2) (at 231.14 80.645 0)
       (effects (font (size 1.27 1.27)) hide)
     )
@@
     (pin "2")
   )
-  (symbol (lib_id "Device:LED") (at 231.14 83.82 0) (mirror x) (unit 1)
-    (in_bom yes) (on_board yes) (fields_autoplaced)
-    (property "Reference" "D5" (id 0) (at 229.5525 77.6945 0))
-    (property "Value" "LED" (id 1) (at 229.5525 80.4696 0))
+  (symbol (lib_id "Device:LED") (at 231.14 83.82 0) (mirror y) (unit 1)
+    (in_bom yes) (on_board yes) (fields_autoplaced)
+    (property "Reference" "D5" (id 0) (at 232.7275 78.5835 0))
+    (property "Value" "LED" (id 1) (at 232.7275 81.3586 0))
     (property "Footprint" "LED_THT:LED_D3.0mm_Horizontal_O1.27mm_Z10.0mm" (id 2) (at 231.14 83.82 0)
       (effects (font (size 1.27 1.27)) hide)
@@
     (in_bom yes) (on_board yes) (fields_autoplaced)
     (property "Reference" "R13" (id 0) (at 213.36 86.4575 90))
-    (property "Value" "1k" (id 1) (at 213.36 89.2326 90))
+    (property "Value" "470" (id 1) (at 213.36 89.2326 90))
     (property "Footprint" "Resistor_THT:R_Axial_DIN0207_L6.3mm_D2.5mm_P7.62mm_Horizontal" (id 2) (at 213.36 93.218 90)
       (effects (font (size 1.27 1.27)) hide)
@@
     )
     (path "/f544f9ba-8782-4d86-bad1-52272bcc53ad"
-      (reference "R13") (unit 1) (value "1k") (footprint "Resistor_THT:R_Axial_DIN0207_L6.3mm_D2.5mm_P7.62mm_Horizontal")
+      (reference "R13") (unit 1) (value "470") (footprint "Resistor_THT:R_Axial_DIN0207_L6.3mm_D2.5mm_P7.62mm_Horizontal")
     )
     (path "/b2bd03a4-ec28-4d74-91f9-acbeba1ad448"

Commit message: Update
Parts:
- R13: value 470 -> 560
Changed lines of the file:
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@@
     (in_bom yes) (on_board yes) (fields_autoplaced)
     (property "Reference" "R13" (id 0) (at 213.36 86.4575 90))
-    (property "Value" "470" (id 1) (at 213.36 89.2326 90))
+    (property "Value" "560" (id 1) (at 213.36 89.2326 90))
     (property "Footprint" "Resistor_THT:R_Axial_DIN0207_L6.3mm_D2.5mm_P7.62mm_Horizontal" (id 2) (at 213.36 93.218 90)
       (effects (font (size 1.27 1.27)) hide)
@@
     )
     (path "/f544f9ba-8782-4d86-bad1-52272bcc53ad"
-      (reference "R13") (unit 1) (value "470") (footprint "Resistor_THT:R_Axial_DIN0207_L6.3mm_D2.5mm_P7.62mm_Horizontal")
+      (reference "R13") (unit 1) (value "560") (footprint "Resistor_THT:R_Axial_DIN0207_L6.3mm_D2.5mm_P7.62mm_Horizontal")
     )
     (path "/b2bd03a4-ec28-4d74-91f9-acbeba1ad448"
