File: Modules/HAGIWO/4Ch Sample Player/Electronics/Main/HAGIWO 4Ch Sampler.kicad_pcb (KiCad board)
At the start: 2 copper layers, 29.2 x 101.6 mm, 48 parts, among them J1 Ch. 1 In, J2 Ch. 3 In, J3 Ch. 2 In, J4 Ch. 4 In, J5 Out, J6 Power, SW1 Left, SW2 Right, SW3 Down, SW4 Mode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

Commit message: Update
Parts:
- removed C2: 1u, Capacitor_SMD:C_0603_1608Metric
- moved R14 1.90 mm to (25.4, 96.5)
Connections:
- J5 pad T: Net-(C2-Pad1) -> Net-(J5-PadT)
- R14 pad 1: Net-(C2-Pad2) -> Net-(J5-PadT)
Routing:
- net Net-(J5-PadT): track 0.00 -> 2.72 mm
- net Net-(C2-Pad1): track 2.70 -> 0.00 mm
- net Net-(C2-Pad2): track 2.57 -> 0.00 mm
- net Net-(R14-Pad2): track 23.6 -> 25.5 mm

Commit message: Update
Parts:
- T1: value 5k -> 20k
