File: Modules/Standard Line/Vactrol VCF/Electronics/Main/Vactrol VCF - Main.kicad_pcb (KiCad board)
At the start: 2 copper layers, 38.1 x 101.6 mm, 41 parts, among them J1 Audio In, J2 Audio Out, J3 Power, J4 CV In, P1 100k, P2 100k, P3 100k, U1 VTL5C, U2 VTL5C, U3 TL072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

Commit message: Update
Parts:
- R10: value 1.4k -> 1.5k
- R2: value 56R -> 47R
Other:
- board text added: "K"
Changed lines of the file:
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@@
   (general
     (thickness 1.6)
-    (drawings 5)
+    (drawings 7)
     (tracks 192)
     (zones 0)
@@
       (effects (font (size 1 1) (thickness 0.15)) (justify mirror))
     )
-    (fp_text value 1.4k (at 3.81 0) (layer F.SilkS)
+    (fp_text value 1.5k (at 3.81 0) (layer F.SilkS)
       (effects (font (size 1 1) (thickness 0.15)))
     )
@@
       (effects (font (size 1 1) (thickness 0.15)) (justify mirror))
     )
-    (fp_text value 56R (at 3.81 0) (layer F.SilkS)
+    (fp_text value 47R (at 3.81 0) (layer F.SilkS)
       (effects (font (size 1 1) (thickness 0.15)))
     )
@@
     )
   )
+  (gr_text K (at 31.75 52.705) (layer F.SilkS)
+    (effects (font (size 1 1) (thickness 0.1)))
+  )
+  (gr_text K (at 31.75 41.275) (layer F.SilkS)
+    (effects (font (size 1 1) (thickness 0.1)))
+  )
   (gr_text "Vactrol VCF\nRev. 012205" (at 21.59 76.2) (layer F.SilkS)
