File: Modules/Standard Line/Manual Gate/Electronics/Control/Manual Gate Control.kicad_pcb (KiCad board)
At the start: 2 copper layers, 19.1 x 101.6 mm, 28 parts, among them J1 Q, J10 Gate, J2 Trigger, J4 /Q, J5 Gate, J6 /Gate, J7 In, J8 In, J9 Q_Qq, SW1 Push

Commit message: Update
Parts:
- R12, R24, R32, R37: value 220k -> 1k

Commit message: Update
Parts:
- removed R12, R24, R32, R37: 1k, Resistor_THT:R_Axial_DIN0207_L6.3mm_D2.5mm_P2.54mm_Vertical
- removed R14: 220k, Resistor_THT:R_Axial_DIN0207_L6.3mm_D2.5mm_P2.54mm_Vertical
- added D1: 1N4733A, Diode_THT:D_DO-35_SOD27_P2.54mm_Vertical_KathodeUp, F.Cu at (17.4, 44.5)
- added D2: 1N4733A, Diode_THT:D_DO-35_SOD27_P2.54mm_Vertical_KathodeUp, F.Cu at (7.87, 63.5)
- added D5: 1N4733A, Diode_THT:D_DO-35_SOD27_P2.54mm_Vertical_KathodeUp, F.Cu at (17.4, 63.5)
- added D7: 1N4733A, Diode_THT:D_DO-35_SOD27_P2.54mm_Vertical_KathodeUp, F.Cu at (7.87, 44.5)
- added D8: 1N4733A, Diode_THT:D_DO-35_SOD27_P2.54mm_Vertical_KathodeUp, F.Cu at (12.6, 82.5)
Other:
- board text added: "Manual Gate Control Rev. 022206"
- board text removed: "Manual Gate Control Rev. 012109"
