File: Modules/Standard Line/Manual Gate/Electronics/Main/Manual Gate Main.kicad_pcb (KiCad board)
At the start: 2 copper layers, 19.1 x 101.6 mm, 59 parts, among them J10 Gate, J3 Power, J8 In, J9 Q_Qq, Q1 BC547, Q10 BC547, Q11 BC547, Q12 BC547, Q2 BC547, Q3 BC547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

Commit message: Update
Parts:
- removed R7: 22k, Resistor_THT:R_Axial_DIN0207_L6.3mm_D2.5mm_P2.54mm_Vertical
- added R1: 100k, Resistor_THT:R_Axial_DIN0207_L6.3mm_D2.5mm_P2.54mm_Vertical, F.Cu at (4.83, 33.0)
- C4: value 100n -> 10n
- R2: value 22k -> 10k
- R25: value 10k -> 220k
- R4: value 22k -> 1k
- R40: value 1M2 -> 1.2M
Routing:
- net Net-(C2-Pad1): track 10.0 -> 17.6 mm
- net Net-(D2-Pad2): track 5.80 -> 2.70 mm
