File: Modules/MFOS/Dual VCA #2/Electronics/Main/Dual VCA #2 Main.kicad_pcb (KiCad board)
At the start: 2 copper layers, 58.4 x 101.6 mm, 63 parts, among them IC1 TL084, IC2 LM13700, J1 Pot #1, J10 SW #2, J11 Sig Out #2, J2 CV In #1, J3 Sig In #1, J4 SW #1, J5 Sig Out #1, J6 Pot #2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

Commit message: Update
Parts:
- removed R41, R42: 1R, Resistor_THT:R_Axial_DIN0207_L6.3mm_D2.5mm_P7.62mm_Horizontal
- added C3: 100n, Capacitor_THT:C_Disc_D3.0mm_W2.0mm_P2.50mm, F.Cu at (27.9, 50.2)
- added C4: 100n, Capacitor_THT:C_Disc_D3.0mm_W2.0mm_P2.50mm, F.Cu at (27.9, 28.6)
- added C5: 100n, Capacitor_THT:C_Disc_D3.0mm_W2.0mm_P2.50mm, F.Cu at (24.1, 81.9)
- added C6: 100n, Capacitor_THT:C_Disc_D3.0mm_W2.0mm_P2.50mm, F.Cu at (29.2, 55.9)
- added D1: 1N5817, Diode_THT:D_DO-41_SOD81_P10.16mm_Horizontal, F.Cu at (17.8, 10.2)
- added D2: 1N5817, Diode_THT:D_DO-41_SOD81_P10.16mm_Horizontal, F.Cu at (33.0, 10.2)
- J7: footprint Connector_IDC:IDC-Header_2x08_P2.54mm_Vertical -> CATs_Eurosynth_Specials:Power_2x5_Vertical
- R11, R31: value 475R -> 470R
- R15, R35: value 499k -> 470k
- R16, R36: value 49k9 -> 47k
- moved C2 27.9 mm to (45.7, 15.2)
- moved C1 25.4 mm to (17.8, 15.2)
- moved J7 13.3 mm to (25.4, 3.81), turned to 270 degrees
Connections:
- IC2 pad 15: Net-(IC2-Pad15) -> (no net)
- IC2 pad 2: Net-(IC2-Pad2) -> (no net)
- J10 pad 1: Net-(J10-Pad1) -> Net-(IC2-Pad16)
- J10 pad 2: Net-(IC2-Pad16) -> Net-(J10-Pad2)
- J4 pad 1: Net-(J4-Pad1) -> Net-(IC2-Pad1)
- J4 pad 2: Net-(IC2-Pad1) -> Net-(J4-Pad2)
- R12 pad 1: Net-(J4-Pad1) -> Net-(J4-Pad2)
- R32 pad 1: Net-(J10-Pad1) -> Net-(J10-Pad2)
Routing:
- net Net-(J10-Pad2): track 0.00 -> 19.7 mm, vias 0 -> 1
- net Net-(J10-Pad1): track 17.1 -> 0.00 mm, vias 1 -> 0
- net -12V: track 203.2 -> 190.0 mm
- net +12VA: track 19.6 -> 8.52 mm
- net +12V: track 189.9 -> 198.3 mm
- net Net-(J4-Pad2): track 0.00 -> 6.69 mm
- net Net-(J4-Pad1): track 5.64 -> 0.00 mm
- net -12VA: track 12.0 -> 8.52 mm
- net Net-(IC2-Pad16): track 34.3 -> 31.7 mm
- net Net-(IC2-Pad1): track 29.2 -> 26.7 mm
