File: Modules/Standard Line/Classic ADSR/Electronics/Main/Classic ADSR Main.kicad_pcb (KiCad board)
At the start: 2 copper layers, 38.1 x 110.5 mm, 53 parts, among them J1 In, J2 Power, J3 OUT, J4 INV OUT, P1 B100K, P2 A100K, P3 A100K, P4 A100K, Q1 MMBT3904, Q2 2N7002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

Commit message: Update
Parts:
- removed G***: LOGO, CATs_Eurosynth_Specials:CATs Tiny
- J2: value Power -> Power_2x5
- J3: value OUT -> ADSR OUT
- R14: value 1k -> 2.4k
