File: Modules/Slim Line/Sample&Hold/Electronics/Main/S&H Main.kicad_pcb (KiCad board)
At the start: 2 copper layers, 38.1 x 101.6 mm, 38 parts, among them J1 Trigger 2, J2 In 2, J3 Trigger 1, J4 In 1, J5 Power, J6 Out 2, J7 Out 1, U1 TL071, U2 LF398, U3 LF398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

Commit message: Update
Parts:
- removed G***: LOGO, Logos:CATs Tiny
- C4, C5: value 22µF -> 10µF
