File: Modules/Slim Line/Sample&Hold/Electronics/Main/S&H Main.kicad_pcb (KiCad board)
At the start: 2 copper layers, 38.1 x 101.6 mm, 37 parts, among them J1 Trigger 2, J2 In 2, J3 Trigger 1, J4 In 1, J5 Power, J6 Out 2, J7 Out 1, U1 TL071, U2 LF398, U3 LF398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

Commit message: Update
Parts:
- added D3: 1N5817, Diode_THT:D_DO-41_SOD81_P10.16mm_Horizontal, F.Cu at (21.6, 78.7)
- added D4: 1N5817, Diode_THT:D_DO-41_SOD81_P10.16mm_Horizontal, F.Cu at (17.8, 96.5)
- added G***: LOGO, CATs_Eurosynth_Specials:CATs Tiny, F.Cu at (33.7, 34.3)
- J5: footprint Connector_IDC:IDC-Header_2x08_P2.54mm_Horizontal -> CATs_Eurosynth_Specials:Power_2x8_Horizontal
- moved C4 23.6 mm to (32.4, 68.6), turned to 0 degrees
- moved C5 1.91 mm to (20.3, 74.3), turned to 180 degrees
- moved J5 0.63 mm to (24.8, 78.7)
Routing:
- net Net-(D4-Pad1): track 0.00 -> 9.52 mm
- net Net-(D3-Pad2): track 0.00 -> 7.88 mm
- net +12V: track 139.8 -> 132.8 mm
- net GND: vias 0 -> 1
Other:
- board text added: "JLCJLCJLCJLC"
- board text added: "Sample&Hold Rev 022212"
- board text removed: "Sample&Hold Rev 010421"
