File: Modules/Slim Line/Buffered Multiple V2/Main/Buffered Multiple V2 Main.kicad_sch (KiCad schematic)
At the start: 49 parts, among them J1 In 1, J2 In 2, J3 Out 1-1, J4 Out 2-1, J5 Out 1-2, J6 Out 2-2, J7 Out 1-3, J8 Out 2-3, J9 Power, U1 TL074CDT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

Commit message: Analog Switch Matrix
Parts:
- C1, C2, C3, C4, C5, C6, C7, C8: LCSC Part # (none) -> C32949
- C10, C11, C13, C14: LCSC Part # (none) -> C307331
- C12, C9: LCSC Part # (none) -> C7171
- D1, D2: LCSC Part # (none) -> C191023
- R1, R11, R12, R13, R14, R17, R18, R19, R2, R20, R3, R4, R5, R6, R7, R8: LCSC Part # (none) -> C25741
- R10, R15, R16, R21, R22, R9: LCSC Part # (none) -> C4410
- U1, U2: LCSC Part # (none) -> C6963
Changed lines of the file:
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@@
+      (effects (font (size 1.27 1.27)) hide)
+    )
+    (property "LCSC Part #" "C6963" (id 5) (at 91.44 41.91 0)
       (effects (font (size 1.27 1.27)) hide)
     )
@@
       (effects (font (size 1.27 1.27)) hide)
     )
+    (property "LCSC Part #" "C32949" (id 5) (at 207.01 100.33 0)
+      (effects (font (size 1.27 1.27)) hide)
+    )
     (pin "1")
     (pin "2")
@@
       (effects (font (size 1.27 1.27)) hide)
     )
+    (property "LCSC Part #" "C4410" (id 5) (at 224.79 41.91 0)
+      (effects (font (size 1.27 1.27)) hide)
+    )
     (pin "1")
     (pin "2")
@@
       (effects (font (size 1.27 1.27)) hide)
     )
+    (property "LCSC Part #" "C6963" (id 5) (at 208.28 76.2 0)
+      (effects (font (size 1.27 1.27)) hide)
+    )
     (pin "12")
     (pin "13")
@@
       (effects (font (size 1.27 1.27)) hide)
     )
+    (property "LCSC Part #" "C4410" (id 5) (at 224.79 76.2 0)
+      (effects (font (size 1.27 1.27)) hide)
+    )
     (pin "1")
     (pin "2")
@@
       (effects (font (size 1.27 1.27)) hide)
     )
+    (property "LCSC Part #" "C25741" (id 5) (at 58.42 31.75 0)
+      (effects (font (size 1.27 1.27)) hide)
+    )
     (pin "1")
     (pin "2")
@@
       (effects (font (size 1.27 1.27)) hide)
     )
+    (property "LCSC Part #" "C6963" (id 5) (at 208.28 41.91 0)
+      (effects (font (size 1.27 1.27)) hide)
+    )
     (pin "5")
     (pin "6")
@@
     )
     (property "LCSC" "C25741" (id 4) (at 191.77 73.66 0)
+      (effects (font (size 1.27 1.27)) hide)
+    )
+    (property "LCSC Part #" "C25741" (id 5) (at 191.77 73.66 0)
       (effects (font (size 1.27 1.27)) hide)
     )
@@
       (effects (font (size 1.27 1.27)) hide)
     )
+    (property "LCSC Part #" "C6963" (id 5) (at 100.33 160.02 0)
+      (effects (font (size 1.27 1.27)) hide)
+    )
     (pin "11")
     (pin "4")
@@
       (effects (font (size 1.27 1.27)) hide)
     )
+    (property "LCSC Part #" "C191023" (id 5) (at 50.8 147.32 0)
+      (effects (font (size 1.27 1.27)) hide)
+    )
     (pin "1")
     (pin "2")
@@
       (effects (font (size 1.27 1.27)) hide)
     )
+    (property "LCSC Part #" "C25741" (id 5) (at 175.26 31.75 0)
+      (effects (font (size 1.27 1.27)) hide)
+    )
     (pin "1")
     (pin "2")
@@
       (effects (font (size 1.27 1.27)) hide)
     )
+    (property "LCSC Part #" "C32949" (id 5) (at 207.01 67.31 0)
+      (effects (font (size 1.27 1.27)) hide)
+    )
     (pin "1")
     (pin "2")
@@
       (effects (font (size 1.27 1.27)) hide)
     )
+    (property "LCSC Part #" "C25741" (id 5) (at 99.06 59.69 0)
+      (effects (font (size 1.27 1.27)) hide)
+    )
     (pin "1")
     (pin "2")
@@
       (effects (font (size 1.27 1.27)) hide)
     )
+    (property "LCSC Part #" "C25741" (id 5) (at 74.93 106.68 0)
+      (effects (font (size 1.27 1.27)) hide)
+    )
     (pin "1")
     (pin "2")
@@
     )
     (property "LCSC" "C307331" (id 4) (at 82.55 166.37 0)
+      (effects (font (size 1.27 1.27)) hide)
+    )
+    (property "LCSC Part #" "C307331" (id 5) (at 82.55 166.37 0)
       (effects (font (size 1.27 1.27)) hide)
     )
@@
       (effects (font (size 1.27 1.27)) hide)
     )
+    (property "LCSC Part #" "C191023" (id 5) (at 50.8 172.72 0)
+      (effects (font (size 1.27 1.27)) hide)
+    )
     (pin "1")
     (pin "2")
@@
       (effects (font (size 1.27 1.27)) hide)
     )
+    (property "LCSC Part #" "C32949" (id 5) (at 90.17 33.02 0)
+      (effects (font (size 1.27 1.27)) hide)
+    )
     (pin "1")
     (pin "2")
@@
     )
     (property "LCSC" "C307331" (id 4) (at 71.12 153.67 0)
+      (effects (font (size 1.27 1.27)) hide)
+    )
+    (property "LCSC Part #" "C307331" (id 5) (at 71.12 153.67 0)
       (effects (font (size 1.27 1.27)) hide)
     )
@@
       (effects (font (size 1.27 1.27)) hide)
     )
+    (property "LCSC Part #" "C25741" (id 5) (at 215.9 25.4 0)
+      (effects (font (size 1.27 1.27)) hide)
+    )
     (pin "1")
     (pin "2")
@@
       (effects (font (size 1.27 1.27)) hide)
     )
+    (property "LCSC Part #" "C32949" (id 5) (at 207.01 33.02 0)
+      (effects (font (size 1.27 1.27)) hide)
+    )
     (pin "1")
     (pin "2")
@@
       (effects (font (size 1.27 1.27)) hide)
     )
+    (property "LCSC Part #" "C4410" (id 5) (at 107.95 76.2 0)
+      (effects (font (size 1.27 1.27)) hide)
+    )
     (pin "1")
     (pin "2")
@@
       (effects (font (size 1.27 1.27)) hide)
     )
+    (property "LCSC Part #" "C32949" (id 5) (at 175.26 22.86 0)
+      (effects (font (size 1.27 1.27)) hide)
+    )
     (pin "1")
     (pin "2")
@@
       (effects (font (size 1.27 1.27)) hide)
     )
+    (property "LCSC Part #" "C32949" (id 5) (at 90.17 100.33 0)
+      (effects (font (size 1.27 1.27)) hide)
+    )
     (pin "1")
     (pin "2")
@@
       (effects (font (size 1.27 1.27)) hide)
     )
+    (property "LCSC Part #" "C25741" (id 5) (at 215.9 59.69 0)
+      (effects (font (size 1.27 1.27)) hide)
+    )
     (pin "1")
     (pin "2")
@@
       (effects (font (size 1.27 1.27)) hide)
     )
+    (property "LCSC Part #" "C25741" (id 5) (at 191.77 106.68 0)
+      (effects (font (size 1.27 1.27)) hide)
+    )
     (pin "1")
     (pin "2")
@@
       (effects (font (size 1.27 1.27)) hide)
     )
+    (property "LCSC Part #" "C4410" (id 5) (at 107.95 41.91 0)
+      (effects (font (size 1.27 1.27)) hide)
+    )
     (pin "1")
     (pin "2")
@@
     )
     (property "LCSC" "C7171" (id 4) (at 57.15 166.37 0)
+      (effects (font (size 1.27 1.27)) hide)
+    )
+    (property "LCSC Part #" "C7171" (id 5) (at 57.15 166.37 0)
       (effects (font (size 1.27 1.27)) hide)
     )
@@
       (effects (font (size 1.27 1.27)) hide)
     )
+    (property "LCSC Part #" "C6963" (id 5) (at 58.42 39.37 0)
+      (effects (font (size 1.27 1.27)) hide)
+    )
     (pin "1")
     (pin "2")
@@
     )
     (property "LCSC" "C32949" (id 4) (at 58.42 22.86 0)
+      (effects (font (size 1.27 1.27)) hide)
+    )
+    (property "LCSC Part #" "C32949" (id 5) (at 58.42 22.86 0)
       (effects (font (size 1.27 1.27)) hide)
     )
@@
       (effects (font (size 1.27 1.27)) hide)
     )
+    (property "LCSC Part #" "C6963" (id 5) (at 109.22 160.02 0)
+      (effects (font (size 1.27 1.27)) hide)
+    )
     (pin "11")
     (pin "4")
@@
       (effects (font (size 1.27 1.27)) hide)
     )
+    (property "LCSC Part #" "C25741" (id 5) (at 41.91 36.83 0)
+      (effects (font (size 1.27 1.27)) hide)
+    )
     (pin "1")
     (pin "2")
@@
       (effects (font (size 1.27 1.27)) hide)
     )
+    (property "LCSC Part #" "C4410" (id 5) (at 224.79 109.22 0)
+      (effects (font (size 1.27 1.27)) hide)
+    )
     (pin "1")
     (pin "2")
@@
       (effects (font (size 1.27 1.27)) hide)
     )
+    (property "LCSC Part #" "C4410" (id 5) (at 107.95 109.22 0)
+      (effects (font (size 1.27 1.27)) hide)
+    )
     (pin "1")
     (pin "2")
@@
       (effects (font (size 1.27 1.27)) hide)
     )
+    (property "LCSC Part #" "C25741" (id 5) (at 74.93 73.66 0)
+      (effects (font (size 1.27 1.27)) hide)
+    )
     (pin "1")
     (pin "2")
@@
       (effects (font (size 1.27 1.27)) hide)
     )
+    (property "LCSC Part #" "C6963" (id 5) (at 91.44 76.2 0)
+      (effects (font (size 1.27 1.27)) hide)
+    )
     (pin "12")
     (pin "13")
@@
       (effects (font (size 1.27 1.27)) hide)
     )
+    (property "LCSC Part #" "C307331" (id 5) (at 71.12 166.37 0)
+      (effects (font (size 1.27 1.27)) hide)
+    )
     (pin "1")
     (pin "2")
@@
       (effects (font (size 1.27 1.27)) hide)
     )
+    (property "LCSC Part #" "C25741" (id 5) (at 99.06 25.4 0)
+      (effects (font (size 1.27 1.27)) hide)
+    )
     (pin "1")
     (pin "2")
@@
       (effects (font (size 1.27 1.27)) hide)
     )
+    (property "LCSC Part #" "C25741" (id 5) (at 215.9 92.71 0)
+      (effects (font (size 1.27 1.27)) hide)
+    )
     (pin "1")
     (pin "2")
@@
     )
     (property "LCSC" "C7171" (id 4) (at 57.15 153.67 0)
+      (effects (font (size 1.27 1.27)) hide)
+    )
+    (property "LCSC Part #" "C7171" (id 5) (at 57.15 153.67 0)
       (effects (font (size 1.27 1.27)) hide)
     )
@@
     )
     (property "LCSC" "C307331" (id 4) (at 82.55 153.67 0)
+      (effects (font (size 1.27 1.27)) hide)
+    )
+    (property "LCSC Part #" "C307331" (id 5) (at 82.55 153.67 0)
       (effects (font (size 1.27 1.27)) hide)
     )
@@
       (effects (font (size 1.27 1.27)) hide)
     )
+    (property "LCSC Part #" "C25741" (id 5) (at 158.75 36.83 0)
+      (effects (font (size 1.27 1.27)) hide)
+    )
     (pin "1")
     (pin "2")
@@
       (effects (font (size 1.27 1.27)) hide)
     )
+    (property "LCSC Part #" "C25741" (id 5) (at 99.06 92.71 0)
+      (effects (font (size 1.27 1.27)) hide)
+    )
     (pin "1")
     (pin "2")
@@
       (effects (font (size 1.27 1.27)) hide)
     )
+    (property "LCSC Part #" "C6963" (id 5) (at 208.28 109.22 0)
+      (effects (font (size 1.27 1.27)) hide)
+    )
     (pin "10")
     (pin "8")
@@
       (effects (font (size 1.27 1.27)) hide)
     )
+    (property "LCSC Part #" "C32949" (id 5) (at 90.17 67.31 0)
+      (effects (font (size 1.27 1.27)) hide)
+    )
     (pin "1")
     (pin "2")
@@
       (effects (font (size 1.27 1.27)) hide)
     )
+    (property "LCSC Part #" "C25741" (id 5) (at 74.93 39.37 0)
+      (effects (font (size 1.27 1.27)) hide)
+    )
     (pin "1")
     (pin "2")
@@
       (effects (font (size 1.27 1.27)) hide)
     )
+    (property "LCSC Part #" "C6963" (id 5) (at 175.26 39.37 0)
+      (effects (font (size 1.27 1.27)) hide)
+    )
     (pin "1")
     (pin "2")
@@
       (effects (font (size 1.27 1.27)) hide)
     )
+    (property "LCSC Part #" "C25741" (id 5) (at 191.77 39.37 0)
+      (effects (font (size 1.27 1.27)) hide)
+    )
     (pin "1")
     (pin "2")
@@
       (effects (font (size 1.27 1.27)) hide)
     )
+    (property "LCSC Part #" "C6963" (id 5) (at 91.44 109.22 0)
+      (effects (font (size 1.27 1.27)) hide)
+    )
