File: Modules/MFOS/Eight Stage Phase Shifter/Electronics/Main/MFOS Eight Stage Phase Shifter - Main.kicad_pcb (KiCad board)
At the start: 2 copper layers, 27.9 x 101.6 mm, 105 parts, among them J1 LFO, J2 CV_OUT, J3 In, J6 Power, Q1 MMBT3904, Q2 MMBT3906, Q3 MMBT3904, U1 TL072, U2 TL072, U3 TL072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

Commit message: Update
Parts:
- D1: value 1N4148W -> 1N4148WS; footprint Diode_SMD:D_SOD-123 -> Diode_SMD:D_SOD-323
- moved D1 1.71 mm to (8.89, 7.62), turned to 0 degrees
Routing:
- net Rate_CW: track 25.9 -> 24.0 mm
Other:
- board text added: "MFOS Phaser Main Rev. 022212"
- board text removed: "MFOS Phaser Main Rev. 012209"
Changed lines of the file:
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@@
     (thickness 1.6)
     (drawings 6)
-    (tracks 704)
+    (tracks 702)
     (zones 0)
     (modules 105)
@@
       (usegerberattributes false)
       (usegerberadvancedattributes true)
-      (creategerberjobfile true)
+      (creategerberjobfile false)
       (excludeedgelayer true)
       (linewidth 0.100000)
@@
       (drillshape 0)
       (scaleselection 1)
-      (outputdirectory "Gerber"))
+      (outputdirectory "Gerber/"))
   )
   (net 0 "")
@@
     (add_net GND)
   )
+  (module Diode_SMD:D_SOD-323 (layer F.Cu)
+    (at 8.89 7.62)
+    (descr SOD-323)
+    (tags SOD-323)
+    (attr smd)
+    (fp_text reference D1 (at 0 -1.85) (layer Dwgs.User) hide
+      (effects (font (size 1 1) (thickness 0.15)))
+    )
+    (fp_text value 1N4148WS (at 0.1 1.9) (layer Dwgs.User) hide
+      (effects (font (size 1 1) (thickness 0.15)))
+    )
+    (fp_line (start -1.5 -0.85) (end 1.05 -0.85) (layer F.SilkS) (width 0.12))
+    (fp_line (start -1.5 0.85) (end 1.05 0.85) (layer F.SilkS) (width 0.12))
+    (fp_line (start -1.6 -0.95) (end -1.6 0.95) (layer F.CrtYd) (width 0.05))
+    (fp_line (start -1.6 0.95) (end 1.6 0.95) (layer F.CrtYd) (width 0.05))
+    (fp_line (start 1.6 -0.95) (end 1.6 0.95) (layer F.CrtYd) (width 0.05))
+    (fp_line (start -1.6 -0.95) (end 1.6 -0.95) (layer F.CrtYd) (width 0.05))
+    (fp_line (start -0.9 -0.7) (end 0.9 -0.7) (layer F.Fab) (width 0.1))
+    (fp_line (start 0.9 -0.7) (end 0.9 0.7) (layer F.Fab) (width 0.1))
+    (fp_line (start 0.9 0.7) (end -0.9 0.7) (layer F.Fab) (width 0.1))
+    (fp_line (start -0.9 0.7) (end -0.9 -0.7) (layer F.Fab) (width 0.1))
+    (fp_line (start -0.3 -0.35) (end -0.3 0.35) (layer F.Fab) (width 0.1))
+    (fp_line (start -0.3 0) (end -0.5 0) (layer F.Fab) (width 0.1))
+    (fp_line (start -0.3 0) (end 0.2 -0.35) (layer F.Fab) (width 0.1))
+    (fp_line (start 0.2 -0.35) (end 0.2 0.35) (layer F.Fab) (width 0.1))
+    (fp_line (start 0.2 0.35) (end -0.3 0) (layer F.Fab) (width 0.1))
+    (fp_line (start 0.2 0) (end 0.45 0) (layer F.Fab) (width 0.1))
+    (fp_line (start -1.5 -0.85) (end -1.5 0.85) (layer F.SilkS) (width 0.12))
+    (fp_text user %R (at 0 -1.85) (layer Dwgs.User) hide
+      (effects (font (size 1 1) (thickness 0.15)))
+    )
+    (pad 2 smd rect (at 1.05 0) (size 0.6 0.45) (layers F.Cu F.Paste F.Mask)
+      (net 53 Rate_CW))
+    (pad 1 smd rect (at -1.05 0) (size 0.6 0.45) (layers F.Cu F.Paste F.Mask)
+      (net 26 "Net-(D1-Pad1)"))
+    (model ${KISYS3DMOD}/Diode_SMD.3dshapes/D_SOD-323.wrl
+      (at (xyz 0 0 0))
+      (scale (xyz 1 1 1))
+      (rotate (xyz 0 0 0))
+    )
+  )
   (module "CATs_Eurosynth_Specials:CATs Tiny" locked (layer B.Cu)
     (at 23.8125 71.12 180)
@@
     )
   )
-  (module Diode_SMD:D_SOD-123 (layer F.Cu)
-    (at 8.255 9.2075 270)
-    (descr SOD-123)
-    (tags SOD-123)
-    (attr smd)
-    (fp_text reference D1 (at 0 -2 90) (layer Dwgs.User) hide
-      (effects (font (size 1 1) (thickness 0.15)))
-    )
-    (fp_text value 1N4148W (at 0 2.1 90) (layer Dwgs.User) hide
-      (effects (font (size 1 1) (thickness 0.15)))
-    )
-    (fp_line (start -2.25 -1) (end -2.25 1) (layer F.SilkS) (width 0.12))
-    (fp_line (start 0.25 0) (end 0.75 0) (layer F.Fab) (width 0.1))
-    (fp_line (start 0.25 0.4) (end -0.35 0) (layer F.Fab) (width 0.1))
-    (fp_line (start 0.25 -0.4) (end 0.25 0.4) (layer F.Fab) (width 0.1))
-    (fp_line (start -0.35 0) (end 0.25 -0.4) (layer F.Fab) (width 0.1))
-    (fp_line (start -0.35 0) (end -0.35 0.55) (layer F.Fab) (width 0.1))
-    (fp_line (start -0.35 0) (end -0.35 -0.55) (layer F.Fab) (width 0.1))
-    (fp_line (start -0.75 0) (end -0.35 0) (layer F.Fab) (width 0.1))
-    (fp_line (start -1.4 0.9) (end -1.4 -0.9) (layer F.Fab) (width 0.1))
-    (fp_line (start 1.4 0.9) (end -1.4 0.9) (layer F.Fab) (width 0.1))
-    (fp_line (start 1.4 -0.9) (end 1.4 0.9) (layer F.Fab) (width 0.1))
-    (fp_line (start -1.4 -0.9) (end 1.4 -0.9) (layer F.Fab) (width 0.1))
-    (fp_line (start -2.35 -1.15) (end 2.35 -1.15) (layer F.CrtYd) (width 0.05))
-    (fp_line (start 2.35 -1.15) (end 2.35 1.15) (layer F.CrtYd) (width 0.05))
-    (fp_line (start 2.35 1.15) (end -2.35 1.15) (layer F.CrtYd) (width 0.05))
-    (fp_line (start -2.35 -1.15) (end -2.35 1.15) (layer F.CrtYd) (width 0.05))
-    (fp_line (start -2.25 1) (end 1.65 1) (layer F.SilkS) (width 0.12))
-    (fp_line (start -2.25 -1) (end 1.65 -1) (layer F.SilkS) (width 0.12))
-    (fp_text user %R (at 0 -2 90) (layer Dwgs.User) hide
-      (effects (font (size 1 1) (thickness 0.15)))
-    )
-    (pad 2 smd rect (at 1.65 0 270) (size 0.9 1.2) (layers F.Cu F.Paste F.Mask)
-      (net 53 Rate_CW))
-    (pad 1 smd rect (at -1.65 0 270) (size 0.9 1.2) (layers F.Cu F.Paste F.Mask)
-      (net 26 "Net-(D1-Pad1)"))
-    (model ${KISYS3DMOD}/Diode_SMD.3dshapes/D_SOD-123.wrl
-      (at (xyz 0 0 0))
-      (scale (xyz 1 1 1))
-      (rotate (xyz 0 0 0))
-    )
-  )
   (module Capacitor_SMD:C_0402_1005Metric (layer F.Cu)
     (at 21.9075 24.4475 270)
@@
     (effects (font (size 0.7 0.7) (thickness 0.08)) (justify left))
   )
-  (gr_text "MFOS Phaser\nMain Rev. 012209" (at 27.305 99.695) (layer B.SilkS)
+  (gr_text "MFOS Phaser\nMain Rev. 022212" (at 27.305 99.695) (layer B.SilkS)
     (effects (font (size 0.8 0.8) (thickness 0.1)) (justify left mirror))
   )
@@
   (via (at 10.16 88.5825) (size 0.8) (drill 0.4) (layers F.Cu B.Cu) (net 1))
   (via (at 6.6675 4.7625) (size 0.8) (drill 0.4) (layers F.Cu B.Cu) (net 1))
-  (via (at 8.255 8.89) (size 0.8) (drill 0.4) (layers F.Cu B.Cu) (net 1))
+  (via (at 8.255 9.398) (size 0.8) (drill 0.4) (layers F.Cu B.Cu) (net 1))
   (via (at 3.4925 64.4525) (size 0.8) (drill 0.4) (layers F.Cu B.Cu) (net 1))
   (via (at 5.715 11.7475) (size 0.8) (drill 0.4) (layers F.Cu B.Cu) (net 1))
@@
   (segment (start 21.11 24.9275) (end 20.955 25.0825) (width 0.2) (layer F.Cu) (net 25))
   (segment (start 21.9075 24.9275) (end 21.11 24.9275) (width 0.2) (layer F.Cu) (net 25))
-  (segment (start 6.225 7.62) (end 6.985 7.62) (width 0.2) (layer F.Cu) (net 26))
-  (segment (start 7.0475 7.5575) (end 6.985 7.62) (width 0.2) (layer F.Cu) (net 26))
-  (segment (start 8.255 7.5575) (end 7.0475 7.5575) (width 0.2) (layer F.Cu) (net 26))
+  (segment (start 6.985 7.62) (end 6.225 7.62) (width 0.2) (layer F.Cu) (net 26))
+  (segment (start 7.84 7.62) (end 6.985 7.62) (width 0.2) (layer F.Cu) (net 26))
   (segment (start 20 88.3125) (end 20 89.215) (width 0.2) (layer F.Cu) (net 27))
   (segment (start 20 89.215) (end 20.32 89.535) (width 0.2) (layer F.Cu) (net 27))
@@
   (segment (start 10.285 14.635) (end 10.315 14.605) (width 0.2) (layer F.Cu) (net 53))
   (segment (start 10.285 16.1925) (end 10.285 14.635) (width 0.2) (layer F.Cu) (net 53))
-  (segment (start 10.315 14.605) (end 8.5725 14.605) (width 0.2) (layer F.Cu) (net 53))
-  (segment (start 8.255 14.2875) (end 8.5725 14.605) (width 0.2) (layer F.Cu) (net 53))
-  (segment (start 8.255 10.8575) (end 8.255 14.2875) (width 0.2) (layer F.Cu) (net 53))
-  (segment (start 2.54 2.54) (end 9.2075 2.54) (width 0.2) (layer F.Cu) (net 53))
-  (segment (start 9.2075 2.54) (end 9.525 2.8575) (width 0.2) (layer F.Cu) (net 53))
-  (segment (start 9.525 2.8575) (end 9.525 10.4775) (width 0.2) (layer F.Cu) (net 53))
-  (segment (start 9.145 10.8575) (end 9.525 10.4775) (width 0.2) (layer F.Cu) (net 53))
-  (segment (start 8.255 10.8575) (end 9.145 10.8575) (width 0.2) (layer F.Cu) (net 53))
+  (segment (start 9.2075 2.54) (end 2.54 2.54) (width 0.2) (layer F.Cu) (net 53))
+  (segment (start 10.5 3.8325) (end 9.2075 2.54) (width 0.2) (layer F.Cu) (net 53))
+  (segment (start 10.5 7.62) (end 10.5 3.8325) (width 0.2) (layer F.Cu) (net 53))
+  (segment (start 10.5 7.62) (end 10.5 12.995) (width 0.2) (layer F.Cu) (net 53))
+  (segment (start 10.315 13.18) (end 10.315 14.605) (width 0.2) (layer F.Cu) (net 53))
+  (segment (start 10.5 12.995) (end 10.315 13.18) (width 0.2) (layer F.Cu) (net 53))
+  (segment (start 9.94 7.62) (end 10.5 7.62) (width 0.2) (layer F.Cu) (net 53))
   (segment (start 13.4 22.5425) (end 12.065 22.5425) (width 0.2) (layer F.Cu) (net 54))
   (segment (start 11.91 22.6975) (end 12.065 22.5425) (width 0.2) (layer F.Cu) (net 54))
