File: Modules/Slim Line/Slimline Clock Divider/Electronics/Main/Slimline Clock Divider SMD Main.kicad_pcb (KiCad board)
At the start: 2 copper layers, 38.1 x 101.6 mm, 43 parts, among them IC1 TL072CDT, IC3 CD4069UBM96, IC4 CD4024BM96, J1 Clock, J2 Out_Div_2, J3 Out_Div_4, J4 Reset, J5 Out_Div_8, J6 Out_Div_16, J7 Power_2x5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

Commit message: Update
Parts:
- removed JP1: Inv_CLK, Jumper:SolderJumper-3_P1.3mm_Bridged2Bar12_RoundedPad1.0x1.5mm
- removed JP2: Inv_RST, Jumper:SolderJumper-3_P1.3mm_Bridged2Bar12_RoundedPad1.0x1.5mm
- removed R13: 1k, Resistor_SMD:R_0603_1608Metric
- added D5: LED, LED_THT:LED_D3.0mm_Horizontal_O3.81mm_Z6.0mm, F.Cu at (5.71, 44.5)
- added D6: LED, LED_THT:LED_D3.0mm_Horizontal_O3.81mm_Z6.0mm, F.Cu at (5.71, 62.2)
- added D7: LED, LED_THT:LED_D3.0mm_Horizontal_O3.81mm_Z6.0mm, F.Cu at (5.71, 80.0)
- added D8: LED, LED_THT:LED_D3.0mm_Horizontal_O3.81mm_Z6.0mm, F.Cu at (5.71, 97.8)
- added D9: 1N4148WS, Diode_SMD:D_SOD-323, F.Cu at (32.6, 15.9)
- added R21: 1k, Resistor_SMD:R_0603_1608Metric, F.Cu at (8.26, 45.7)
- added R22: 1k, Resistor_SMD:R_0603_1608Metric, F.Cu at (8.26, 63.5)
- added R23: 1k, Resistor_SMD:R_0603_1608Metric, F.Cu at (8.26, 81.3)
- added R24: 1k, Resistor_SMD:R_0603_1608Metric, F.Cu at (8.26, 99.1)
- D3: value LED -> 1N4148WS; footprint LED_THT:LED_D3.0mm_Horizontal_O3.81mm_Z6.0mm -> Diode_SMD:D_SOD-323
- moved G*** 57.1 mm to (31.8, 63.5)
- moved R19 47.7 mm to (10.2, 99.1), turned to 90 degrees
- moved R20 43.5 mm to (12.1, 99.1)
- moved R17 30.4 mm to (10.2, 81.3), turned to 90 degrees
- moved R18 26.2 mm to (12.1, 81.3)
- moved D3 24.3 mm to (19.1, 22.9), turned to 180 degrees
- moved J2 21.1 mm to (0.00, 36.8)
- moved R8 16.3 mm to (12.1, 45.7)
- moved J3 15.9 mm to (0.00, 54.6)
- moved R7 13.7 mm to (10.2, 45.7), turned to 90 degrees
- moved R14 13.6 mm to (10.2, 63.5), turned to 90 degrees
- moved J5 10.8 mm to (0.00, 72.4)
- moved R4 10.6 mm to (15.9, 6.99)
- moved R16 10.5 mm to (12.1, 63.5)
- moved R10 9.94 mm to (15.9, 20.3)
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Connections:
- net Net-(Q1-Pad2) renamed L/2
- net Net-(Q2-Pad2) renamed L/4
- net Net-(Q3-Pad2) renamed L/8
- net Net-(Q4-Pad2) renamed L/16
- D3 pad 1: GND -> Net-(IC3-Pad1)
- D3 pad 2: Net-(D3-Pad2) -> Net-(IC1-Pad1)
- IC3 pad 1: Net-(IC1-Pad1) -> Net-(IC3-Pad1)
- IC3 pad 3: Net-(IC3-Pad2) -> (no net)
- IC3 pad 4: Net-(IC3-Pad4) -> (no net)
- IC3 pad 5: Net-(IC1-Pad7) -> Net-(IC3-Pad5)
- IC4 pad 1: Net-(IC4-Pad1) -> Net-(IC3-Pad2)
- IC4 pad 2: Net-(IC4-Pad2) -> Net-(IC3-Pad8)
Routing:
- net Net-(IC1-Pad7): track 74.6 -> 3.94 mm, vias 5 -> 0
- net L/16: track 2.42 -> 71.2 mm
- net Net-(J6-PadT): track 69.0 -> 9.35 mm
- net Net-(IC3-Pad5): track 0.00 -> 57.5 mm, vias 0 -> 5
- net L/8: track 2.42 -> 49.0 mm
- net Net-(J5-PadT): track 51.8 -> 9.35 mm
- net Net-(IC4-Pad2): track 34.6 -> 0.00 mm, vias 3 -> 0
- net Net-(J3-PadT): track 32.8 -> 9.35 mm
- net Net-(IC3-Pad2): track 5.79 -> 28.7 mm, vias 1 -> 2
- net L/4: track 2.42 -> 24.8 mm
- net Net-(IC4-Pad1): track 21.3 -> 0.00 mm, vias 1 -> 0
- net Net-(IC3-Pad8): track 4.79 -> 24.4 mm, vias 1 -> 2
- net L/2: track 2.42 -> 16.3 mm
- net Net-(IC1-Pad5): track 26.7 -> 15.0 mm
- net Net-(J1-PadT): track 1.99 -> 13.2 mm
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Other:
- board text added: "Clock Divider Rev. 032302"
- board text removed: "Clock Divider Rev. 022301"
