File: Modules/Slim Line/Slimline Clock Divider/Electronics/Main/Slimline Clock Divider SMD Main.kicad_sch (KiCad schematic)
At the start: 42 parts, among them IC1 TL072CDT, IC3 CD4069UBM96, IC4 CD4024BM96, J1 Clock, J2 Out_Div_2, J3 Out_Div_4, J4 Reset, J5 Out_Div_8, J6 Out_Div_16, J7 Power_2x5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

Commit message: Update
Parts:
- removed D3: LED, LED_THT:LED_D3.0mm_Horizontal_O3.81mm_Z6.0mm, symbol Device:LED
- removed unit 2 of IC3
- removed JP1: Inv_CLK, Jumper:SolderJumper-3_P1.3mm_Bridged2Bar12_RoundedPad1.0x1.5mm, symbol Jumper:SolderJumper_3_Bridged12
- removed JP2: Inv_RST, Jumper:SolderJumper-3_P1.3mm_Bridged2Bar12_RoundedPad1.0x1.5mm, symbol Jumper:SolderJumper_3_Bridged12
- removed R13: 1k, Resistor_SMD:R_0603_1608Metric, symbol Device:R
- added D3, D9: 1N4148WS, Diode_SMD:D_SOD-323, symbol Diode:1N4148WS
- added D5, D6, D7, D8: LED, LED_THT:LED_D3.0mm_Horizontal_O3.81mm_Z6.0mm, symbol Device:LED
- added R21, R22, R23, R24: 1k, Resistor_SMD:R_0603_1608Metric, symbol Device:R
Connections:
- net GND: now also D5.1 (K), D6.1 (K), D7.1 (K), D8.1 (K)
- net at IC1.7: now also D9.2 (A); no longer IC3.5
- net L/4: now reaches Q2.2 (E), R14.1
- net L/4: now also R22.1
- net at R14.2, R16.1: no longer J3.T
- net L/16: now reaches Q4.2 (E), R19.1
- net L/16: now also R24.1
- net at IC3.8: now also IC4.2 (MR)
- net at IC1.1, R12.1: now also D3.2 (A); no longer IC3.1
- net at IC3.2: now also IC4.1 (~{CP})
- net L/2: now reaches Q1.2 (E), R7.1
- net L/2: now also R21.1
- net L/8: now reaches Q3.2 (E), R17.1
- net L/8: now also R23.1
- new net: D8.2 (A), R24.2
- new net: D5.2 (A), R21.2
- new net: D7.2 (A), R23.2
- new net: D9.1 (K), IC3.5
- new net: D6.2 (A), R22.2
- new net: D3.1 (K), IC3.1
