File: Modules/Slim Line/Sample&Hold SMD/Electronics/Front/Sample_and_Hold Front.kicad_pcb (KiCad board)
At the start: 2 copper layers, 9.8 x 128.5 mm, 8 parts

Commit message: Update
Other:
- net class Default removed
