File: Modules/Slim Line/Sample&Hold SMD/Electronics/Main/Sample_and_Hold SMD Main.kicad_pcb (KiCad board)
At the start: 2 copper layers, 38.1 x 101.6 mm, 42 parts, among them J1 Trigger 2, J2 In 2, J3 Trigger 1, J4 In 1, J5 Power, J6 Out 2, J7 Out 1, U1 OP07CDR, U2 LF398, U3 LF398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

Commit message: Update
Other:
- net class Default removed

Commit message: Update
Parts:
- added REF**: WEEE-Logo_4.2x6mm_SilkScreen, Symbol:WEEE-Logo_4.2x6mm_SilkScreen, F.Cu at (34.3, 68.6)
- added REF**: CE-Logo_8.5x6mm_SilkScreen, Symbol:CE-Logo_8.5x6mm_SilkScreen, F.Cu at (26.7, 68.6)
Other:
- board text removed: "JLCJLCJLCJLC"
